File: ROV_PCIe_USB_HUB_FE1.1S/power.kicad_sch (KiCad schematic)
At the start: 18 parts, among them U3 TPS62A02APDDC, U4 TPS62A02APDDC

Commit message: updates
Parts:
- C27: Part Number CL05C100JB5NNNC -> CL05C100JB5NNNC; now not fitted; now left out of the parts list
- C28, C32: footprint Capacitor_SMD:C_1206_3216Metric -> Capacitor_SMD:C_0805_2012Metric; Part Number CL31B226MPHNNNE -> CL21A226MOQNNNE
- C29, C33: Part Number CL21A106KOQNNNE -> CL21A106KOQNNNE
- C30, C34: Part Number CL05B104KB5NNNC -> CL05B104KO5NNNC
- C31: Part Number CL05C220JB5NNNC -> CL05C180JB5NNNC; now not fitted; now left out of the parts list
- R13, R16: Part Number AC0603FR-0710KL -> RC0603FR-0710KL
- R14: Part Number AC0603FR-07453KL -> RC0603FR-07453KL
- R15, R18: Part Number AC0603FR-07100KL -> RC0603FR-07100KL
- R17: Part Number AC0603FR-0775KL -> RC0603FR-0775KL
Changed lines of the file:
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@@
 			)
 		)
-		(property "Part Number" "AC0603FR-07453KL"
+		(property "Part Number" "RC0603FR-07453KL"
 			(at 151.13 71.12 0)
 			(hide yes)
@@
 			)
 		)
-		(property "Part Number" "CL05B104KB5NNNC"
+		(property "Part Number" "CL05B104KO5NNNC"
 			(at 106.68 77.47 0)
 			(hide yes)
@@
 			)
 		)
-		(property "Footprint" "Capacitor_SMD:C_1206_3216Metric"
+		(property "Footprint" "Capacitor_SMD:C_0805_2012Metric"
 			(at 175.26 120.65 0)
 			(hide yes)
@@
 			)
 		)
-		(property "Part Number" "CL31B226MPHNNNE"
+		(property "Part Number" "CL21A226MOQNNNE"
 			(at 175.26 120.65 0)
 			(hide yes)
@@
 			)
 		)
-		(property "Part Number" "AC0603FR-0710KL"
+		(property "Part Number" "RC0603FR-0710KL"
 			(at 130.81 105.41 0)
 			(hide yes)
@@
 			)
 		)
-		(property "Footprint" "Capacitor_SMD:C_1206_3216Metric"
+		(property "Footprint" "Capacitor_SMD:C_0805_2012Metric"
 			(at 175.26 74.93 0)
 			(hide yes)
@@
 			)
 		)
-		(property "Part Number" "CL31B226MPHNNNE"
+		(property "Part Number" "CL21A226MOQNNNE"
 			(at 175.26 74.93 0)
 			(hide yes)
@@
 			)
 		)
-		(property "Part Number" "AC0603FR-07100KL"
+		(property "Part Number" "RC0603FR-07100KL"
 			(at 151.13 124.46 0)
 			(hide yes)
@@
 			)
 		)
-		(property "Part Number" "CL21A106KOQNNNE"
+		(property "Part Number" "CL21A106KOQNNNE "
 			(at 101.6 77.47 0)
 			(hide yes)
@@
 			)
 		)
-		(property "Part Number" "AC0603FR-0710KL"
+		(property "Part Number" "RC0603FR-0710KL"
 			(at 130.81 57.15 0)
 			(hide yes)
@@
 			)
 		)
-		(property "Part Number" "AC0603FR-0775KL"
+		(property "Part Number" "RC0603FR-0775KL"
 			(at 151.13 116.84 0)
 			(hide yes)
@@
 		(body_style 1)
 		(exclude_from_sim no)
-		(in_bom yes)
+		(in_bom no)
 		(on_board yes)
 		(in_pos_files yes)
-		(dnp no)
+		(dnp yes)
 		(fields_autoplaced yes)
 		(property "Reference" "C27"
@@
 			)
 		)
-		(property "Part Number" "CL05C100JB5NNNC"
+		(property "Part Number" "CL05C100JB5NNNC "
 			(at 162.56 71.12 0)
 			(hide yes)
@@
 		(body_style 1)
 		(exclude_from_sim no)
-		(in_bom yes)
+		(in_bom no)
 		(on_board yes)
 		(in_pos_files yes)
-		(dnp no)
+		(dnp yes)
 		(fields_autoplaced yes)
 		(property "Reference" "C31"
@@
 			)
 		)
-		(property "Part Number" "CL05C220JB5NNNC"
+		(property "Part Number" "CL05C180JB5NNNC "
 			(at 162.56 116.84 0)
 			(hide yes)
@@
 			)
 		)
-		(property "Part Number" "AC0603FR-07100KL"
+		(property "Part Number" "RC0603FR-07100KL"
 			(at 151.13 78.74 0)
 			(hide yes)
@@
 			)
 		)
-		(property "Part Number" "CL21A106KOQNNNE"
+		(property "Part Number" "CL21A106KOQNNNE "
 			(at 101.6 123.19 0)
 			(hide yes)
@@
 			)
 		)
-		(property "Part Number" "CL05B104KB5NNNC"
+		(property "Part Number" "CL05B104KO5NNNC"
 			(at 106.68 123.19 0)
 			(hide yes)
