File: ROV_PCIe_USB_HUB_FE1.1S/rov_usb.kicad_pcb (KiCad board)
At the start: 4 copper layers, 55.5 x 68.5 mm, 123 parts, among them J1 525591652, J2 61400826021, J3 691311500102, J4 692121430000, J5 61400826021, J6 61400826021, J7 629722000214, U1 UPD720201K8-701-BAC-A, U10 TPS2051CDBV, U11 MIC5504-3.3YM5, U12 TPS2116DRL, U2 SST25VF512A-33-4C-SAE, U3 TPS62A02APDDC, U4 TPS62A02APDDC, U5 TPS2051CDBV, U6 TPS2051CDBV, U7 FE1.1S-BQFN24B, U8 TS3USB30EDGSR, U9 TPS2051CDBV, Y1 ABM8-24.000MHZ-B2-T, Y2 ABM8-12.000MHZ-B2-T

Commit message: updates
Parts:
- C21, C28, C32, C9: footprint Capacitor_SMD:C_1206_3216Metric -> Capacitor_SMD:C_0805_2012Metric
- C44, C46, C47: footprint Capacitor_SMD:C_0805_2012Metric -> Capacitor_SMD:C_0603_1608Metric
- J3: renamed from J2; value 61400826021 -> USB-A-D-RA
- J4: value 692121430000 -> USB-A3-S-VT-CS5A
- J5, J6: value 61400826021 -> USB-A-D-RA
- R12: value 1k6 1% -> 1k6
- R29: renamed from R23; value 2k7 1% -> 2k7
- U10, U5, U6, U9: value TPS2051CDBV -> TPS2051CDBVR
- U11: value MIC5504-3.3YM5 -> MIC5504-3.3YM5-TR
- moved C9 0.51 mm to (207.7, 151.9)
- renumbered D7 to D1, D4 to D10, D5 to D11, D8 to D2, D9 to D3, D12 to D4, D10 to D5, D11 to D6, D1 to D7, D2 to D8, D3 to D9, J3 to J2, R31 to R19, R32 to R20, R33 to R21, R36 to R22, R34 to R23, R35 to R24, R19 to R25, R20 to R26, R21 to R27, R22 to R28, R24 to R30, R25 to R31, R26 to R32, R27 to R33, R28 to R34, R29 to R35
Routing:
- net GND: track 137.8 -> 135.8 mm, vias 116 -> 115
- net +3.3V: track 124.8 -> 126.3 mm
- net +5V: track 51.5 -> 52.3 mm
