File: ROV_PCIe_USB_HUB_FE1.1S/rov_usb.kicad_sch (KiCad schematic)
At the start: 9 parts, among them J1 525591652

Commit message: updates
Parts:
- C1, C2: Part Number CL05B104KB5NNNC -> CL05B104KO5NNNC
- R1: Part Number AC0603FR-073K6L -> RC0603FR-073K6L
- R2: Part Number AC0603FR-07100KL -> RC0603FR-07100KL
- R3: Part Number AC0603FR-076K8L -> RC0603FR-076K8L
Changed lines of the file:
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@@
 			)
 		)
-		(property "Part Number" "AC0603FR-07100KL"
+		(property "Part Number" "RC0603FR-07100KL"
 			(at 71.12 82.55 0)
 			(hide yes)
@@
 			)
 		)
-		(property "Part Number" "CL05B104KB5NNNC"
+		(property "Part Number" "CL05B104KO5NNNC"
 			(at 162.56 72.39 90)
 			(hide yes)
@@
 			)
 		)
-		(property "Part Number" "AC0603FR-076K8L"
+		(property "Part Number" "RC0603FR-076K8L"
 			(at 74.93 82.55 0)
 			(hide yes)
@@
 			)
 		)
-		(property "Part Number" "AC0603FR-073K6L"
+		(property "Part Number" "RC0603FR-073K6L"
 			(at 74.93 62.23 0)
 			(hide yes)
@@
 			)
 		)
-		(property "Part Number" "CL05B104KB5NNNC"
+		(property "Part Number" "CL05B104KO5NNNC"
 			(at 162.56 76.2 90)
 			(hide yes)
