File: ROV_PCIe_USB_HUB_FE1.1S/usb.kicad_sch (KiCad schematic)
At the start: 57 parts, among them J2 61400826021, J3 691311500102, J4 692121430000, J5 61400826021, J6 61400826021, J7 629722000214, U10 TPS2051CDBV, U11 MIC5504-3.3YM5, U12 TPS2116DRL, U5 TPS2051CDBV, U6 TPS2051CDBV, U7 FE1.1S-BQFN24B, U8 TS3USB30EDGSR, U9 TPS2051CDBV, Y2 ABM8-12.000MHZ-B2-T

Commit message: updates
Parts:
- C35, C36, C37, C38, C41, C42, C43, C45: Part Number CL21A106KOQNNNE -> CL21A106KOQNNNE
- C39, C40: Part Number CL05B104KB5NNNC -> CL05B104KO5NNNC
- C44, C46, C47: footprint Capacitor_SMD:C_0805_2012Metric -> Capacitor_SMD:C_0603_1608Metric; Part Number CL21B105KOFNNNE -> CL10B105KO8NNNC
- J3: renamed from J2; value 61400826021 -> USB-A-D-RA; Part Number 61400826021 -> USB-A-D-RA
- J4: value 692121430000 -> USB-A3-S-VT-CS5A; Part Number 692121430000 -> USB-A3-S-VT-CS5A
- J5, J6: value 61400826021 -> USB-A-D-RA; Part Number 61400826021 -> USB-A-D-RA
- R19: renamed from R31; Part Number AC0603FR-07470RL -> RC0603FR-07270RL
- R20: renamed from R32; Part Number AC0603FR-07470RL -> RC0603FR-07270RL
- R21: renamed from R33; Part Number AC0603FR-07470RL -> RC0603FR-07270RL
- R22: renamed from R36; Part Number AC0603FR-07470RL -> RC0603FR-07100RL
- R23: renamed from R34; Part Number AC0603FR-07470RL -> RC0603FR-07270RL
- R24: renamed from R35; Part Number AC0603FR-07470RL -> RC0603FR-07100RL
- R25: renamed from R19; Part Number AC0603FR-0710KL -> RC0603FR-0710KL
- R26: renamed from R20; Part Number AC0603FR-07100KL -> RC0603FR-07100KL
- R27: renamed from R21; Part Number AC0603FR-07470RL -> RC0603FR-07470RL
- R28: renamed from R22; Part Number AC0603FR-07470RL -> RC0603FR-07470RL
- R29: renamed from R23; value 2k7 1% -> 2k7; Part Number RT0603BRD072K7L -> RC0603FR-072K7L
- R30: renamed from R24; Part Number AC0603FR-075K1L -> RC0603FR-075K1L
- R31: renamed from R25; Part Number AC0603FR-075K1L -> RC0603FR-075K1L
- R32: renamed from R26; Part Number AC0603FR-07470RL -> RC0603FR-07470RL
- R33: renamed from R27; Part Number AC0603FR-07330KL -> RC0603FR-07330KL
- R34: renamed from R28; Part Number AC0603FR-07100KL -> RC0603FR-07100KL
- R35: renamed from R29; Part Number AC0603FR-07100KL -> RC0603FR-07100KL
- U10, U5, U6, U9: value TPS2051CDBV -> TPS2051CDBVR; Part Number TPS2051CDBV -> TPS2051CDBVR
- U11: value MIC5504-3.3YM5 -> MIC5504-3.3YM5-TR; Part Number MIC5504-3.3YM5 -> MIC5504-3.3YM5-TR
- renumbered D7 to D1, D4 to D10, D5 to D11, D8 to D2, D9 to D3, D12 to D4, D10 to D5, D11 to D6, D1 to D7, D2 to D8, D3 to D9, J3 to J2
