File: ROV_PCIe_Adapter/ROV_PCIe_Adapter.kicad_pcb (KiCad board)
At the start: 4 copper layers, 20.3 x 28.3 mm, 16 parts, among them J1 Bus_PCI_Express_x1, J2 525591652, U1 TPS563201

Commit message: changes
Parts:
- added C10: 100n, Capacitor_SMD:C_0402_1005Metric, F.Cu at (160.2, 82.0)
- added C7: 22u, Capacitor_SMD:C_0805_2012Metric, F.Cu at (158.0, 106.0)
- added C8: 100n, Capacitor_SMD:C_0402_1005Metric, F.Cu at (156.5, 106.8)
- added C9: 22u, Capacitor_SMD:C_0805_2012Metric, F.Cu at (158.5, 82.2)
- moved G*** 10.9 mm to (171.0, 95.8)
Routing:
- net GND: track 48.4 -> 58.3 mm, vias 29 -> 35
- net +12V: track 18.9 -> 20.6 mm

Commit message: changes
Parts:
- added R5: 0R, Resistor_SMD:R_0402_1005Metric, F.Cu at (164.5, 92.1)
- C5: value 22u -> 10p; footprint Capacitor_SMD:C_0805_2012Metric -> Capacitor_SMD:C_0402_1005Metric
- C7: value 22u -> 10u
- F1: value MF-MSMF110/16-2 -> MF-MSMF150/12X-2
- moved C5 8.92 mm to (165.5, 96.7)
- moved C4 1.72 mm to (161.7, 88.5)
- moved R3 1.00 mm to (165.8, 98.0)
- moved R4 1.00 mm to (165.8, 99.5)
- moved C9 0.56 mm to (158.0, 82.5)
- moved C3 0.36 mm to (162.6, 92.1)
- moved R2 0.30 mm to (163.9, 90.5)
- moved R1 0.30 mm to (160.8, 90.5)
Connections:
- C3 pad 2: Net-(U1-VBST) -> Net-(C3-Pad2)
- C5 pad 2: GND -> Net-(U1-VFB)
Routing:
- net Net-(U1-VFB): track 2.79 -> 6.02 mm
- net Net-(U1-VBST): track 3.02 -> 1.49 mm
- net GND: track 58.3 -> 57.0 mm, vias 35 -> 32
- net +5V: track 11.1 -> 10.0 mm
- net Net-(C3-Pad2): track 0.00 -> 0.94 mm
- net /PCIE_PWR_EN: track 17.2 -> 16.5 mm

Commit message: final
Parts:
- added D1: LED, LED_SMD:LED_0603_1608Metric, F.Cu at (164.5, 102.0)
- added D2: LED, LED_SMD:LED_0603_1608Metric, F.Cu at (156.5, 99.5)
- added R6: 5k1, Resistor_SMD:R_0603_1608Metric, F.Cu at (166.0, 102.0)
- added R7: 1k6, Resistor_SMD:R_0603_1608Metric, F.Cu at (158.0, 99.5)
- C4, C9: footprint Capacitor_SMD:C_0805_2012Metric -> Capacitor_SMD:C_1206_3216Metric
- moved C9 0.25 mm to (158.0, 82.8)
Routing:
- net GND: track 57.0 -> 63.1 mm, vias 32 -> 39
- net +3.3V_AUX: track 4.05 -> 0.00 mm, vias 1 -> 0
- net +12V: track 20.6 -> 22.8 mm
- net +5V: track 10.0 -> 11.8 mm
- net Net-(D1-K): track 0.00 -> 1.53 mm
- net Net-(D2-K): track 0.00 -> 1.51 mm
Other:
- board text added: "+12V"
- board text added: "+5V"
