File: ROV_PCIe_USB_HUB_USB2514/power.kicad_sch (KiCad schematic)
At the start: 18 parts, among them U3 TPS62A02APDDC, U4 TPS62A02APDDC

Commit message: updates
Parts:
- C27, C31: now not fitted; now left out of the parts list
- C28, C32: footprint Capacitor_SMD:C_1206_3216Metric -> Capacitor_SMD:C_0805_2012Metric; Part Number CL31B226MPHNNNE -> CL21A226MOQNNNE
- C29, C33: Part Number CL21A106KOQNNNE -> CL21A106KOQNNNE
- C30, C34: Part Number CL05B104KB5NNNC -> CL05B104KO5NNNC
- R13, R16: Part Number AC0603FR-0710KL -> RC0603FR-0710KL
- R14: Part Number AC0603FR-07453KL -> RC0603FR-07453KL
- R15, R18: Part Number AC0603FR-07100KL -> RC0603FR-07100KL
- R17: Part Number AC0603FR-0775KL -> RC0603FR-0775KL
Changed lines of the file:
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@@
 			)
 		)
-		(property "Part Number" "AC0603FR-07453KL"
+		(property "Part Number" "RC0603FR-07453KL"
 			(at 151.13 71.12 0)
 			(hide yes)
@@
 			)
 		)
-		(property "Part Number" "CL05B104KB5NNNC"
+		(property "Part Number" "CL05B104KO5NNNC"
 			(at 106.68 77.47 0)
 			(hide yes)
@@
 			)
 		)
-		(property "Footprint" "Capacitor_SMD:C_1206_3216Metric"
+		(property "Footprint" "Capacitor_SMD:C_0805_2012Metric"
 			(at 175.26 120.65 0)
 			(hide yes)
@@
 			)
 		)
-		(property "Part Number" "CL31B226MPHNNNE"
+		(property "Part Number" "CL21A226MOQNNNE"
 			(at 175.26 120.65 0)
 			(hide yes)
@@
 			)
 		)
-		(property "Part Number" "AC0603FR-0710KL"
+		(property "Part Number" "RC0603FR-0710KL"
 			(at 130.81 105.41 0)
 			(hide yes)
@@
 			)
 		)
-		(property "Footprint" "Capacitor_SMD:C_1206_3216Metric"
+		(property "Footprint" "Capacitor_SMD:C_0805_2012Metric"
 			(at 175.26 74.93 0)
 			(hide yes)
@@
 			)
 		)
-		(property "Part Number" "CL31B226MPHNNNE"
+		(property "Part Number" "CL21A226MOQNNNE"
 			(at 175.26 74.93 0)
 			(hide yes)
@@
 			)
 		)
-		(property "Part Number" "AC0603FR-07100KL"
+		(property "Part Number" "RC0603FR-07100KL"
 			(at 151.13 124.46 0)
 			(hide yes)
@@
 			)
 		)
-		(property "Part Number" "CL21A106KOQNNNE"
+		(property "Part Number" "CL21A106KOQNNNE "
 			(at 101.6 77.47 0)
 			(hide yes)
@@
 			)
 		)
-		(property "Part Number" "AC0603FR-0710KL"
+		(property "Part Number" "RC0603FR-0710KL"
 			(at 130.81 57.15 0)
 			(hide yes)
@@
 			)
 		)
-		(property "Part Number" "AC0603FR-0775KL"
+		(property "Part Number" "RC0603FR-0775KL"
 			(at 151.13 116.84 0)
 			(hide yes)
@@
 		(body_style 1)
 		(exclude_from_sim no)
-		(in_bom yes)
+		(in_bom no)
 		(on_board yes)
 		(in_pos_files yes)
-		(dnp no)
+		(dnp yes)
 		(fields_autoplaced yes)
 		(property "Reference" "C27"
@@
 		(body_style 1)
 		(exclude_from_sim no)
-		(in_bom yes)
+		(in_bom no)
 		(on_board yes)
 		(in_pos_files yes)
-		(dnp no)
+		(dnp yes)
 		(fields_autoplaced yes)
 		(property "Reference" "C31"
@@
 			)
 		)
-		(property "Part Number" "AC0603FR-07100KL"
+		(property "Part Number" "RC0603FR-07100KL"
 			(at 151.13 78.74 0)
 			(hide yes)
@@
 			)
 		)
-		(property "Part Number" "CL21A106KOQNNNE"
+		(property "Part Number" "CL21A106KOQNNNE "
 			(at 101.6 123.19 0)
 			(hide yes)
@@
 			)
 		)
-		(property "Part Number" "CL05B104KB5NNNC"
+		(property "Part Number" "CL05B104KO5NNNC"
 			(at 106.68 123.19 0)
 			(hide yes)

Commit message: changes
Parts:
- C28, C32: footprint Capacitor_SMD:C_0805_2012Metric -> Capacitor_SMD:C_1206_3216Metric; Part Number CL21A226MOQNNNE -> CC1206KKX5R8BB226
- C29, C33: Part Number CL21A106KOQNNNE -> CC0805KRX5R8BB106
- C30, C34: Part Number CL05B104KO5NNNC -> CC0402KRX7R8BB104
Changed lines of the file:
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@@
 			)
 		)
-		(property "Part Number" "CL05B104KO5NNNC"
+		(property "Part Number" "CC0402KRX7R8BB104"
 			(at 106.68 77.47 0)
 			(hide yes)
@@
 			)
 		)
-		(property "Footprint" "Capacitor_SMD:C_0805_2012Metric"
+		(property "Footprint" "Capacitor_SMD:C_1206_3216Metric"
 			(at 175.26 120.65 0)
 			(hide yes)
@@
 			)
 		)
-		(property "Part Number" "CL21A226MOQNNNE"
+		(property "Part Number" "CC1206KKX5R8BB226"
 			(at 175.26 120.65 0)
 			(hide yes)
@@
 			)
 		)
-		(property "Footprint" "Capacitor_SMD:C_0805_2012Metric"
+		(property "Footprint" "Capacitor_SMD:C_1206_3216Metric"
 			(at 175.26 74.93 0)
 			(hide yes)
@@
 			)
 		)
-		(property "Part Number" "CL21A226MOQNNNE"
+		(property "Part Number" "CC1206KKX5R8BB226"
 			(at 175.26 74.93 0)
 			(hide yes)
@@
 			)
 		)
-		(property "Part Number" "CL21A106KOQNNNE "
+		(property "Part Number" "CC0805KRX5R8BB106"
 			(at 101.6 77.47 0)
 			(hide yes)
@@
 			)
 		)
-		(property "Part Number" "CL21A106KOQNNNE "
+		(property "Part Number" "CC0805KRX5R8BB106"
 			(at 101.6 123.19 0)
 			(hide yes)
@@
 			)
 		)
-		(property "Part Number" "CL05B104KO5NNNC"
+		(property "Part Number" "CC0402KRX7R8BB104"
 			(at 106.68 123.19 0)
 			(hide yes)

Commit message: final
Parts:
- renumbered R13 to R14, R14 to R15, R15 to R16, R16 to R17, R17 to R18, R18 to R19
Changed lines of the file:
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@@
 		(dnp no)
 		(fields_autoplaced yes)
-		(property "Reference" "R14"
+		(property "Reference" "R15"
 			(at 153.67 69.8499 0)
 			(show_name no)
@@
 			(project "rov_usb"
 				(path "/e63e39d7-6ac0-4ffd-8aa3-1841a4541b55/894a28e8-d816-4717-bdb5-e6633a8bfe56"
-					(reference "R14")
+					(reference "R15")
 					(unit 1)
 				)
@@
 		(in_pos_files yes)
 		(dnp no)
-		(property "Reference" "#PWR017"
+		(property "Reference" "#PWR019"
 			(at 130.81 55.88 0)
 			(hide yes)
@@
 			(project "rov_usb"
 				(path "/e63e39d7-6ac0-4ffd-8aa3-1841a4541b55/894a28e8-d816-4717-bdb5-e6633a8bfe56"
-					(reference "#PWR017")
+					(reference "#PWR019")
 					(unit 1)
 				)
@@
 		(in_pos_files yes)
 		(dnp no)
-		(property "Reference" "#PWR024"
+		(property "Reference" "#PWR026"
 			(at 119.38 135.89 0)
 			(hide yes)
@@
 			(project "rov_usb"
 				(path "/e63e39d7-6ac0-4ffd-8aa3-1841a4541b55/894a28e8-d816-4717-bdb5-e6633a8bfe56"
-					(reference "#PWR024")
+					(reference "#PWR026")
 					(unit 1)
 				)
@@
 		(in_pos_files yes)
 		(dnp no)
-		(property "Reference" "R16"
+		(property "Reference" "R17"
 			(at 133.35 104.1399 0)
 			(show_name no)
@@
 			(project "rov_usb"
 				(path "/e63e39d7-6ac0-4ffd-8aa3-1841a4541b55/894a28e8-d816-4717-bdb5-e6633a8bfe56"
-					(reference "R16")
+					(reference "R17")
 					(unit 1)
 				)
@@
 		(dnp no)
 		(fields_autoplaced yes)
-		(property "Reference" "R18"
+		(property "Reference" "R19"
 			(at 153.67 123.1899 0)
 			(show_name no)
@@
 			(project "rov_usb"
 				(path "/e63e39d7-6ac0-4ffd-8aa3-1841a4541b55/894a28e8-d816-4717-bdb5-e6633a8bfe56"
-					(reference "R18")
+					(reference "R19")
 					(unit 1)
 				)
@@
 		(in_pos_files yes)
 		(dnp no)
-		(property "Reference" "#PWR022"
+		(property "Reference" "#PWR024"
 			(at 106.68 113.03 0)
 			(hide yes)
@@
 			(project "rov_usb"
 				(path "/e63e39d7-6ac0-4ffd-8aa3-1841a4541b55/894a28e8-d816-4717-bdb5-e6633a8bfe56"
-					(reference "#PWR022")
+					(reference "#PWR024")
 					(unit 1)
 				)
@@
 		(in_pos_files yes)
 		(dnp no)
-		(property "Reference" "#PWR018"
+		(property "Reference" "#PWR020"
 			(at 106.68 67.31 0)
 			(hide yes)
@@
 			(project "rov_usb"
 				(path "/e63e39d7-6ac0-4ffd-8aa3-1841a4541b55/894a28e8-d816-4717-bdb5-e6633a8bfe56"
-					(reference "#PWR018")
+					(reference "#PWR020")
 					(unit 1)
 				)
@@
 		(in_pos_files yes)
 		(dnp no)
-		(property "Reference" "#PWR020"
+		(property "Reference" "#PWR022"
 			(at 119.38 90.17 0)
 			(hide yes)
@@
 			(project "rov_usb"
 				(path "/e63e39d7-6ac0-4ffd-8aa3-1841a4541b55/894a28e8-d816-4717-bdb5-e6633a8bfe56"
-					(reference "#PWR020")
+					(reference "#PWR022")
 					(unit 1)
 				)
@@
 		(in_pos_files yes)
 		(dnp no)
-		(property "Reference" "R13"
+		(property "Reference" "R14"
 			(at 133.35 55.8799 0)
 			(show_name no)
@@
 			(project "rov_usb"
 				(path "/e63e39d7-6ac0-4ffd-8aa3-1841a4541b55/894a28e8-d816-4717-bdb5-e6633a8bfe56"
-					(reference "R13")
+					(reference "R14")
 					(unit 1)
 				)
@@
 		(dnp no)
 		(fields_autoplaced yes)
-		(property "Reference" "R17"
+		(property "Reference" "R18"
 			(at 153.67 115.5699 0)
 			(show_name no)
@@
 			(project "rov_usb"
 				(path "/e63e39d7-6ac0-4ffd-8aa3-1841a4541b55/894a28e8-d816-4717-bdb5-e6633a8bfe56"
-					(reference "R17")
+					(reference "R18")
 					(unit 1)
 				)
@@
 		(dnp no)
 		(fields_autoplaced yes)
-		(property "Reference" "R15"
+		(property "Reference" "R16"
 			(at 153.67 77.4699 0)
 			(show_name no)
@@
 			(project "rov_usb"
 				(path "/e63e39d7-6ac0-4ffd-8aa3-1841a4541b55/894a28e8-d816-4717-bdb5-e6633a8bfe56"
-					(reference "R15")
+					(reference "R16")
 					(unit 1)
 				)
@@
 		(in_pos_files yes)
 		(dnp no)
-		(property "Reference" "#PWR019"
+		(property "Reference" "#PWR021"
 			(at 175.26 68.58 0)
 			(hide yes)
@@
 			(project "rov_usb"
 				(path "/e63e39d7-6ac0-4ffd-8aa3-1841a4541b55/894a28e8-d816-4717-bdb5-e6633a8bfe56"
-					(reference "#PWR019")
+					(reference "#PWR021")
 					(unit 1)
 				)
@@
 		(in_pos_files yes)
 		(dnp no)
-		(property "Reference" "#PWR021"
+		(property "Reference" "#PWR023"
 			(at 130.81 104.14 0)
 			(hide yes)
@@
 			(project "rov_usb"
 				(path "/e63e39d7-6ac0-4ffd-8aa3-1841a4541b55/894a28e8-d816-4717-bdb5-e6633a8bfe56"
-					(reference "#PWR021")
+					(reference "#PWR023")
 					(unit 1)
 				)
@@
 		(in_pos_files yes)
 		(dnp no)
-		(property "Reference" "#PWR023"
+		(property "Reference" "#PWR025"
 			(at 175.26 114.3 0)
 			(hide yes)
@@
 			(project "rov_usb"
 				(path "/e63e39d7-6ac0-4ffd-8aa3-1841a4541b55/894a28e8-d816-4717-bdb5-e6633a8bfe56"
-					(reference "#PWR023")
+					(reference "#PWR025")
 					(unit 1)
 				)
