File: ROV_PCIe_USB_HUB_USB2514/rov_usb.kicad_pcb (KiCad board)
At the start: 4 copper layers, 55.5 x 68.5 mm, 128 parts, among them J1 525591652, J2 61400826021, J3 691311500102, J4 692121430000, J5 61400826021, J6 61400826021, J7 629722000214, U1 UPD720201K8-701-BAC-A, U10 TPS2051CDBV, U11 MIC5504-3.3YM5, U12 TPS2116DRL, U13 USB2514B_Bi, U2 SST25VF512A-33-4C-SAE, U3 TPS62A02APDDC, U4 TPS62A02APDDC, U5 TPS2051CDBV, U6 TPS2051CDBV, U8 TS3USB30EDGSR, U9 TPS2051CDBV, Y1 ABM8-24.000MHZ-B2-T, Y3 ABM8-24.000MHZ-B2-T

Commit message: updates
Parts:
- C21, C28, C32, C9: footprint Capacitor_SMD:C_1206_3216Metric -> Capacitor_SMD:C_0805_2012Metric
- C48: renamed from C49; value 18p -> 27p
- C49: renamed from C48; value 18p -> 27p
- C54: renamed from C44; footprint Capacitor_SMD:C_0805_2012Metric -> Capacitor_SMD:C_0603_1608Metric
- C56: renamed from C46; footprint Capacitor_SMD:C_0805_2012Metric -> Capacitor_SMD:C_0603_1608Metric
- C57: renamed from C47; footprint Capacitor_SMD:C_0805_2012Metric -> Capacitor_SMD:C_0603_1608Metric
- J3: renamed from J2; value 61400826021 -> USB-A-D-RA
- J4: value 692121430000 -> USB-A3-S-VT-CS5A
- J5, J6: value 61400826021 -> USB-A-D-RA
- R12: value 1k6 1% -> 1k6
- R21: renamed from R37; value 12.0k 1% -> 12k
- U10, U5, U6, U9: value TPS2051CDBV -> TPS2051CDBVR
- U11: value MIC5504-3.3YM5 -> MIC5504-3.3YM5-TR
- U8: renamed from U13; value USB2514B_Bi -> USB2514B/M2
- moved C9 0.51 mm to (207.5, 151.9)
- renumbered C60 to C36, C59 to C37, C58 to C38, C57 to C39, C53 to C40, C54 to C41, C55 to C42, C36 to C43, C37 to C44, C40 to C45, C41 to C46, C52 to C47, C42 to C51, C51 to C52, C43 to C53, C45 to C55, D7 to D1, D8 to D2, D9 to D3, D12 to D4, D10 to D5, D11 to D6, FB3 to FB2, J3 to J2, R38 to R19, R19 to R20, R30 to R22, R24 to R23, R26 to R24, R27 to R26, R28 to R27, R31 to R28, R32 to R29, R29 to R30, R33 to R31, R36 to R32, R34 to R33, R35 to R34, U8 to U7, Y3 to Y2
Routing:
- net +3.3V: track 123.0 -> 124.8 mm
- net GND: track 131.1 -> 129.7 mm, vias 121 -> 120
- net +5V: track 51.5 -> 52.6 mm

Commit message: updates (fe1.1s board deprecated)
Parts:
- removed H2: MountingHole, MountingHole:MountingHole_3.2mm_M3
- added D7: SMAJ5.0A, Diode_SMD:D_SMA, F.Cu at (218.6, 104.2)
- added D8: BZX84C10, Diode_SMD:D_0402_1005Metric, F.Cu at (210.6, 101.0)
- added G***: LOGO, LOGO, B.Cu at (400.6, 260.6)
- added Q1: AO3401A, Package_TO_SOT_SMD:SOT-23, F.Cu at (214.9, 102.6)
- added R35: 100k, Resistor_SMD:R_0603_1608Metric, F.Cu at (212.3, 102.1)
- added R36: 5k1, Resistor_SMD:R_0603_1608Metric, F.Cu at (204.2, 122.8)
- added U13: USBLC6-2SC6, Package_TO_SOT_SMD:SOT-23-6, F.Cu at (218.0, 129.1)
- added U14: USBLC6-2SC6, Package_TO_SOT_SMD:SOT-23-6, F.Cu at (218.0, 125.7)
- added U15: USBLC6-2SC6, Package_TO_SOT_SMD:SOT-23-6, F.Cu at (228.8, 111.5)
- added U16: USBLC6-2SC6, Package_TO_SOT_SMD:SOT-23-6, F.Cu at (225.3, 111.5)
- added U17: USBLC6-2SC6, Package_TO_SOT_SMD:SOT-23-6, F.Cu at (217.5, 141.9)
- added U18: USBLC6-2SC6, Package_TO_SOT_SMD:SOT-23-6, F.Cu at (217.5, 145.3)
- added U19: USBLC6-2SC6, Package_TO_SOT_SMD:SOT-23-6, F.Cu at (195.5, 100.2)
- added U20: USBLC6-2SC6, Package_TO_SOT_SMD:SOT-23-6, F.Cu at (185.8, 128.1)
- added U21: TPD4E05U06DQA, Package_SON:USON-10_2.5x1.0mm_P0.5mm, F.Cu at (195.9, 131.6)
- moved U9 23.1 mm to (232.8, 113.9), turned to -90 degrees
- moved U10 21.5 mm to (236.3, 113.8), turned to -90 degrees
- moved C51 19.2 mm to (232.8, 110.8), turned to 180 degrees
- moved C53 17.3 mm to (236.3, 110.8), turned to 180 degrees
- moved J6 10.8 mm to (233.0, 106.7), turned to 180 degrees
- moved C46 9.76 mm to (218.9, 136.2)
- moved U6 9.76 mm to (215.8, 136.2)
- moved R34 7.87 mm to (221.1, 111.1)
- moved D6 7.87 mm to (218.0, 111.1)
- moved D5 3.44 mm to (210.4, 106.9)
- moved R33 3.44 mm to (213.6, 106.9)
- moved J5 3.38 mm to (222.8, 131.4)
- moved R22 3.02 mm to (205.2, 114.4)
- moved R24 3.02 mm to (205.2, 115.9)
- moved C43 2.68 mm to (218.9, 132.7)
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Connections:
- J2 pad 2: VBUS -> Net-(D7-A1)
- R20 pad 2: /USB/USBC_VBUS -> Net-(U7-S)
- U7 pad 1: /USB/USBC_VBUS -> Net-(U7-S)
Routing:
- net VBUS: track 23.9 -> 60.5 mm, vias 7 -> 12
- net GND: track 129.7 -> 146.7 mm, vias 120 -> 147
- net Net-(J5B-VBUS): track 9.71 -> 26.6 mm, vias 0 -> 1
- net /USB/FE_DP3: track 15.3 -> 29.2 mm
- net /USB/FE_DN3: track 15.5 -> 29.3 mm
- net /USB/FE_DN1: track 12.5 -> 26.1 mm
- net /USB/FE_DP1: track 12.5 -> 26.1 mm
- net /USB/FE_DN2: track 15.1 -> 28.3 mm
- net /USB/FE_DP2: track 15.1 -> 28.3 mm
- net /USB/~{OVC2}: track 17.8 -> 29.8 mm
- net /USB/EN2: track 14.6 -> 25.1 mm
- net /USB/FE_3V3: track 30.0 -> 40.1 mm, vias 6 -> 7
- net Net-(J6B-VBUS): track 27.5 -> 18.0 mm, vias 0 -> 2
- net /USB/FE_DN4: track 12.8 -> 21.4 mm
- net /USB/FE_DP4: track 12.8 -> 21.3 mm
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- added copper zone on F.Cu, net Net-(D7-A1)
Other:
- board text added: "+"
- board text added: "-"
- board text added: "EXT_VBUS"
- board text removed: "1 2 3 4 A"
- board text removed: "VBUS"

Commit message: changes
Parts:
- C21, C28, C32, C9: footprint Capacitor_SMD:C_0805_2012Metric -> Capacitor_SMD:C_1206_3216Metric
- R1: value 3k6 -> 5k1
- R12: value 1k6 -> 1k6 1%
- R21: value 12k -> 12k 1%
- R26: value 330k -> 10k
- R3: value 6k8 -> 10k
- R30: value 100k -> 5k1
- moved G*** 6.15 mm to (209.4, 130.5) (x2)
- moved C32 1.08 mm to (194.9, 117.2)
- moved C28 1.06 mm to (195.3, 109.2)
- moved C9 0.34 mm to (207.7, 151.6)
- moved C21 0.21 mm to (206.7, 137.3)
Routing:
- net GND: track 146.7 -> 155.1 mm, vias 147 -> 152
- net +1.05V: track 58.1 -> 51.1 mm, vias 11 -> 13
- net +3.3V: track 124.8 -> 118.5 mm, vias 16 -> 18
- added copper zone on F.Cu, net +1.05V
- added copper zone on F.Cu, net +3.3V

Commit message: final
Parts:
- J8: renamed from J7; value 629722000214 -> USB4085-GF-A
- Q1: value AO3401A -> DMP3013SFV; footprint Package_TO_SOT_SMD:SOT-23 -> Package_SON:Diodes_PowerDI3333-8
- U21: renamed from U12; value TPS2116DRL -> TPS2116DRLR
- U9: renamed from U21; value TPD4E05U06DQA -> TPD4E05U06DQAR
- moved D2 7.31 mm to (214.2, 107.2)
- moved R4 6.31 mm to (216.0, 107.2)
- moved R35 3.47 mm to (210.5, 105.2), turned to 0 degrees
- moved Q1 0.42 mm to (214.5, 102.8)
- renumbered D7 to D1, D8 to D2, D1 to D3, D2 to D4, D3 to D5, D4 to D6, D5 to D7, D6 to D8, H3 to H2, J3 to J4, J4 to J5, J5 to J6, J6 to J7, R9 to R10, R10 to R11, R11 to R12, R12 to R13, R13 to R14, R14 to R15, R15 to R16, R16 to R17, R17 to R18, R18 to R19, R19 to R20, R36 to R21, R20 to R22, R21 to R23, R22 to R24, R23 to R25, R24 to R26, R25 to R27, R26 to R28, R27 to R29, R28 to R30, R29 to R31, R30 to R32, R31 to R33, R32 to R34, R33 to R35, R34 to R36, R35 to R4, R4 to R5, R5 to R6, R6 to R7, R7 to R8, R8 to R9, U17 to U10, U6 to U11, U14 to U12, U7 to U13, U8 to U14, U9 to U15, U15 to U16, U19 to U17, U10 to U18, U16 to U19, U11 to U20, U20 to U5, U18 to U6, U5 to U7, U13 to U8
Connections:
- D1 pad 1: Net-(D7-A1) -> Net-(D1-A1)
- D2 pad 2: Net-(D8-A) -> Net-(D2-A)
- J2 pad 2: Net-(D7-A1) -> Net-(D1-A1)
- Q1 pad 1: Net-(D8-A) -> VBUS
- Q1 pad 3: Net-(D7-A1) -> VBUS
- R4 pad 1: Net-(D8-A) -> Net-(D2-A)
Routing:
- net GND: track 155.1 -> 173.1 mm, vias 152 -> 153
- net VBUS: track 60.5 -> 43.1 mm, vias 12 -> 14
- net Net-(D8-A): track 4.34 -> 0.00 mm
- net Net-(D2-A): track 0.00 -> 4.33 mm
- added copper zone on F.Cu, net Net-(D1-A1)
- added copper zone on F.Cu, net VBUS
- removed copper zone on F.Cu, net Net-(D7-A1)
