File: ROV_PCIe_USB_HUB_USB2514/rov_usb.kicad_pcb (KiCad board)
At the start: 4 copper layers, 55.5 x 68.5 mm, 142 parts, among them J1 525591652, J2 691311500102, J4 USB-A-D-RA, J5 USB-A3-S-VT-CS5A, J6 USB-A-D-RA, J7 USB-A-D-RA, J8 USB4085-GF-A, Q1 DMP3013SFV, U1 UPD720201K8-701-BAC-A, U10 USBLC6-2SC6, U11 TPS2051CDBVR, U12 USBLC6-2SC6, U13 TS3USB30EDGSR, U14 USB2514B/M2, U15 TPS2051CDBVR, U16 USBLC6-2SC6, U17 USBLC6-2SC6, U18 TPS2051CDBVR, U19 USBLC6-2SC6, U2 SST25VF512A-33-4C-SAE, U20 MIC5504-3.3YM5-TR, U21 TPS2116DRLR, U3 TPS62A02APDDC, U4 TPS62A02APDDC, U5 USBLC6-2SC6, U6 USBLC6-2SC6, U7 TPS2051CDBVR, U8 USBLC6-2SC6, U9 TPD4E05U06DQAR, Y1 ABM8-24.000MHZ-B2-T, Y2 ABM8-24.000MHZ-B2-T

Commit message: changes
Parts:
- moved G*** 107.5 mm to (293.1, 259.6)
Changed lines of the file:
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@@
 	(footprint "LOGO"
 		(layer "B.Cu")
-		(at 400.65 260.6 180)
+		(at 293.144106 259.60612 180)
 		(property "Reference" "G***"
 			(at 0.070366 0.036709 0)

Commit message: move parts to project specific libs
Parts:
- removed J1: 525591652, snadol:525591652
- added J9: 525591652, ROV_PCIe_USB_HUB:525591652, F.Cu at (185.8, 142.7)
- Q1: value DMP3013SFV -> DMP3018SFV
- U1: value UPD720201K8-701-BAC-A -> UPD720201K8-7x1-BAC-A; footprint snadol:QFN68_8X8_REN -> ROV_PCIe_USB_HUB:QFN-68-1EP_8x8mm_P0.4mm_EP6.2x6.2mm
- U2: footprint snadol:SST25VF512A -> Package_SO:SOIC-8_3.9x4.9mm_P1.27mm
- moved U2 0.21 mm to (193.5, 151.7)
Routing:
- net +3.3V: track 118.5 -> 120.1 mm
- net Net-(U1-SPISCK): track 11.4 -> 12.7 mm
- net GND: track 173.1 -> 173.3 mm, vias 153 -> 137
