File: ROV_PCIe_USB_HUB_USB2514/rov_usb.kicad_sch (KiCad schematic)
At the start: 14 parts, among them J1 525591652, J2 691311500102, J3 691351500002, Q1 DMP3018SFV

Commit message: move parts to project specific libs
Parts:
- removed J1: 525591652, snadol:525591652, symbol snadol:525591652
- added J9: 525591652, ROV_PCIe_USB_HUB:525591652, symbol ROV_PCIe_USB_HUB:525591652
Connections:
- net +5V: now also J9.1, J9.2
- net GND: now also J9.12, J9.3, J9.6, J9.9
- net PCIE_CLKREQ_N: now also J9.15
- net PCIE_DET_WAKE: now also J9.14
- net PCIE_PWR_EN: now also J9.13
- net PCIE_RST_B: now also J9.16
- net PI_PCIE_CLK_N: now also J9.5
- net PI_PCIE_CLK_P: now also J9.4
- net PI_PCIE_RX_N: now also J9.8
- net PI_PCIE_RX_P: now also J9.7
- net PI_PCIE_TX_N: now also J9.11
- net PI_PCIE_TX_P: now also J9.10
Changed lines of the file:
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@@
-	)
-	(symbol
-		(lib_id "snadol:525591652")
-		(at 43.18 39.37 0)
-		(mirror y)
-		(unit 1)
-		(body_style 1)
-		(exclude_from_sim no)
-		(in_bom yes)
-		(on_board yes)
-		(in_pos_files yes)
-		(dnp no)
-		(fields_autoplaced yes)
-		(property "Reference" "J1"
-			(at 29.21 57.1499 0)
-			(show_name no)
-			(do_not_autoplace no)
-			(effects
-				(font
-					(size 1.524 1.524)
-				)
-				(justify left)
-			)
-		)
-		(property "Value" "525591652"
-			(at 29.21 59.6899 0)
-			(show_name no)
-			(do_not_autoplace no)
-			(effects
-				(font
-					(size 1.524 1.524)
-				)
-				(justify left)
-			)
-		)
-		(property "Footprint" "snadol:525591652"
-			(at 43.18 39.37 0)
-			(hide yes)
-			(show_name no)
-			(do_not_autoplace no)
-			(effects
-				(font
-					(size 1.27 1.27)
-					(italic yes)
-				)
-			)
-		)
-		(property "Datasheet" "https://www.molex.com/en-us/products/part-detail-pdf/525591652?display=pdf"
-			(at 43.18 39.37 0)
-			(hide yes)
-			(show_name no)
-			(do_not_autoplace no)
-			(effects
-				(font
-					(size 1.27 1.27)
-					(italic yes)
-				)
-			)
-		)
-		(property "Description" ""
-			(at 43.18 39.37 0)
-			(hide yes)
-			(show_name no)
-			(do_not_autoplace no)
-			(effects
-				(font
-					(size 1.27 1.27)
-				)
-			)
-		)
-		(property "KLC_S3.3" ""
-			(at 43.18 39.37 0)
-			(hide yes)
-			(show_name no)
-			(do_not_autoplace no)
-			(effects
-				(font
-					(size 1.27 1.27)
-				)
-			)
-		)
-		(property "KLC_S4.1" ""
-			(at 43.18 39.37 0)
-			(hide yes)
-			(show_name no)
-			(do_not_autoplace no)
-			(effects
-				(font
-					(size 1.27 1.27)
-				)
-			)
-		)
-		(property "Part Number" "525591652"
-			(at 43.18 39.37 0)
-			(hide yes)
-			(show_name no)
-			(do_not_autoplace no)
-			(effects
-				(font
-					(size 1.27 1.27)
-				)
-			)
-		)
-		(pin "8"
-		)
-		(pin "10"
-		)
-		(pin "13"
-		)
-		(pin "12"
-		)
-		(pin "4"
-		)
-		(pin "2"
-		)
-		(pin "5"
-		)
-		(pin "1"
-		)
-		(pin "15"
-		)
-		(pin "3"
-		)
-		(pin "6"
-		)
-		(pin "7"
-		)
-		(pin "9"
-		)
-		(pin "11"
-		)
-		(pin "16"
-		)
-		(pin "14"
-		)
-		(instances
-			(project "rov_usb"
-				(path "/e63e39d7-6ac0-4ffd-8aa3-1841a4541b55"
-					(reference "J1")
-					(unit 1)
-				)
-			)
-		)
 	)
 	(symbol
@@
 					(unit 1)
 				)
+			)
+		)
+	)
+	(symbol
+		(lib_id "ROV_PCIe_USB_HUB:525591652")
+		(at 38.1 36.83 0)
+		(mirror y)
+		(unit 1)
+		(body_style 1)
+		(exclude_from_sim no)
+		(in_bom yes)
+		(on_board yes)
+		(in_pos_files yes)
+		(dnp no)
+		(fields_autoplaced yes)
+		(property "Reference" "J9"
+			(at 34.29 31.75 0)
+			(show_name no)
+			(do_not_autoplace no)
+			(effects
+				(font
+					(size 1.524 1.524)
+				)
+			)
+		)
+		(property "Value" "525591652"
+			(at 34.29 34.29 0)
+			(show_name no)
+			(do_not_autoplace no)
+			(effects
+				(font
+					(size 1.524 1.524)
+				)
+			)
+		)
+		(property "Footprint" "ROV_PCIe_USB_HUB:525591652"
+			(at 34.544 87.122 0)
+			(hide yes)
+			(show_name no)
+			(do_not_autoplace no)
+			(effects
+				(font
+					(size 1.27 1.27)
+					(italic yes)
+				)
+			)
+		)
+		(property "Datasheet" "https://www.molex.com/en-us/products/part-detail-pdf/525591652?display=pdf"
+			(at 34.29 84.328 0)
+			(hide yes)
+			(show_name no)
+			(do_not_autoplace no)
+			(effects
+				(font
+					(size 1.27 1.27)
+					(italic yes)
+				)
+			)
+		)
+		(property "Description" ""
+			(at 43.18 39.37 0)
+			(hide yes)
+			(show_name no)
+			(do_not_autoplace no)
+			(effects
+				(font
+					(size 1.27 1.27)
+				)
+			)
+		)
+		(pin "14"
+		)
+		(pin "1"
+		)
+		(pin "2"
+		)
+		(pin "3"
+		)
+		(pin "11"
+		)
+		(pin "7"
+		)
+		(pin "10"
+		)
+		(pin "5"
+		)
+		(pin "13"
+		)
+		(pin "16"
+		)
+		(pin "6"
+		)
+		(pin "4"
+		)
+		(pin "9"
+		)
+		(pin "8"
+		)
+		(pin "12"
+		)
+		(pin "15"
+		)
+		(instances
+			(project "rov_usb"
+				(path "/e63e39d7-6ac0-4ffd-8aa3-1841a4541b55"
+					(reference "J9")
+					(unit 1)
+				)
