File: ROV_PCIe_USB_HUB_USB2514/pcie_usb.kicad_sch (KiCad schematic)
At the start: 37 parts, among them U1 UPD720201K8-701-BAC-A, U2 SST25VF512A-33-4C-SAE, Y1 ABM8-24.000MHZ-B2-T

Commit message: updates
Parts:
- C10: Part Number CL21A106KOQNNNE -> CL21A106KOQNNNE
- C11, C12, C13, C14, C15, C16, C17, C18, C19, C20, C22, C23, C3, C4, C5, C6, C7, C8: Part Number CL05B104KB5NNNC -> CL05B104KO5NNNC
- C21, C9: footprint Capacitor_SMD:C_1206_3216Metric -> Capacitor_SMD:C_0805_2012Metric; Part Number CL31B226MPHNNNE -> CL21A226MOQNNNE
- C24, C25: Part Number CL05C270JB51PNC -> CL05C270JB5NNNC
- R10, R4, R5, R6, R7, R8: Part Number AC0603FR-0710KL -> RC0603FR-0710KL
- R11: Part Number AC0402FR-070RL -> RC0402JR-070RL
- R12: value 1k6 1% -> 1k6; Part Number RT0603BRD071K6L -> RC0603FR-071K6L
- R9: Part Number AC0603FR-07100KL -> RC0603FR-07100KL
Changed lines of the file:
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@@
 			)
 		)
-		(property "Part Number" "AC0603FR-0710KL"
+		(property "Part Number" "RC0603FR-0710KL"
 			(at 107.95 116.84 0)
 			(hide yes)
@@
 			)
 		)
-		(property "Part Number" "CL05B104KB5NNNC"
+		(property "Part Number" "CL05B104KO5NNNC"
 			(at 29.21 29.21 0)
 			(hide yes)
@@
 			)
 		)
-		(property "Part Number" "AC0603FR-07100KL"
+		(property "Part Number" "RC0603FR-07100KL"
 			(at 81.28 115.57 0)
 			(hide yes)
@@
 			)
 		)
-		(property "Part Number" "CL05B104KB5NNNC"
+		(property "Part Number" "CL05B104KO5NNNC"
 			(at 39.37 46.99 0)
 			(hide yes)
@@
 			)
 		)
-		(property "Part Number" "CL05B104KB5NNNC"
+		(property "Part Number" "CL05B104KO5NNNC"
 			(at 91.44 59.69 90)
 			(hide yes)
@@
 			)
 		)
-		(property "Part Number" "AC0402FR-070RL"
+		(property "Part Number" "RC0402JR-070RL"
 			(at 114.3 129.54 90)
 			(hide yes)
@@
 			)
 		)
-		(property "Part Number" "AC0603FR-0710KL"
+		(property "Part Number" "RC0603FR-0710KL"
 			(at 85.09 96.52 0)
 			(hide yes)
@@
 			)
 		)
-		(property "Part Number" "CL05C270JB51PNC"
+		(property "Part Number" "CL05C270JB5NNNC"
 			(at 95.25 127 90)
 			(hide yes)
@@
 			)
 		)
-		(property "Part Number" "CL05B104KB5NNNC"
+		(property "Part Number" "CL05B104KO5NNNC"
 			(at 34.29 29.21 0)
 			(hide yes)
@@
 			)
 		)
-		(property "Part Number" "CL05B104KB5NNNC"
+		(property "Part Number" "CL05B104KO5NNNC"
 			(at 64.77 46.99 0)
 			(hide yes)
@@
 			)
 		)
-		(property "Footprint" "Capacitor_SMD:C_1206_3216Metric"
+		(property "Footprint" "Capacitor_SMD:C_0805_2012Metric"
 			(at 64.77 29.21 0)
 			(hide yes)
@@
 			)
 		)
-		(property "Part Number" "CL31B226MPHNNNE"
+		(property "Part Number" "CL21A226MOQNNNE"
 			(at 64.77 29.21 0)
 			(hide yes)
@@
 			)
 		)
-		(property "Part Number" "CL05B104KB5NNNC"
+		(property "Part Number" "CL05B104KO5NNNC"
 			(at 49.53 29.21 0)
 			(hide yes)
@@
 			)
 		)
-		(property "Part Number" "CL05B104KB5NNNC"
+		(property "Part Number" "CL05B104KO5NNNC"
 			(at 34.29 46.99 0)
 			(hide yes)
@@
 			)
 		)
-		(property "Part Number" "CL05C270JB51PNC"
+		(property "Part Number" "CL05C270JB5NNNC"
 			(at 95.25 134.62 90)
 			(hide yes)
@@
 			)
 		)
-		(property "Part Number" "CL05B104KB5NNNC"
+		(property "Part Number" "CL05B104KO5NNNC"
 			(at 223.52 39.37 0)
 			(hide yes)
@@
 			)
 		)
-		(property "Part Number" "AC0603FR-0710KL"
+		(property "Part Number" "RC0603FR-0710KL"
 			(at 77.47 96.52 0)
 			(hide yes)
@@
 			)
 		)
-		(property "Footprint" "Capacitor_SMD:C_1206_3216Metric"
+		(property "Footprint" "Capacitor_SMD:C_0805_2012Metric"
 			(at 73.66 46.99 0)
 			(hide yes)
@@
 			)
 		)
-		(property "Part Number" "CL31B226MPHNNNE"
+		(property "Part Number" "CL21A226MOQNNNE"
 			(at 73.66 46.99 0)
 			(hide yes)
@@
 			)
 		)
-		(property "Part Number" "CL05B104KB5NNNC"
+		(property "Part Number" "CL05B104KO5NNNC"
 			(at 59.69 46.99 0)
 			(hide yes)
@@
 			)
 		)
-		(property "Part Number" "CL05B104KB5NNNC"
+		(property "Part Number" "CL05B104KO5NNNC"
 			(at 49.53 46.99 0)
 			(hide yes)
@@
 			)
 		)
-		(property "Part Number" "AC0603FR-0710KL"
+		(property "Part Number" "RC0603FR-0710KL"
 			(at 73.66 96.52 0)
 			(hide yes)
@@
 			)
 		)
-		(property "Part Number" "CL05B104KB5NNNC"
+		(property "Part Number" "CL05B104KO5NNNC"
 			(at 44.45 46.99 0)
 			(hide yes)
@@
 			)
 		)
-		(property "Part Number" "CL05B104KB5NNNC"
+		(property "Part Number" "CL05B104KO5NNNC"
 			(at 91.44 62.23 90)
 			(hide yes)
@@
 			)
 		)
-		(property "Part Number" "CL21A106KOQNNNE"
+		(property "Part Number" "CL21A106KOQNNNE "
 			(at 213.36 39.37 0)
 			(hide yes)
@@
 			)
 		)
-		(property "Part Number" "CL05B104KB5NNNC"
+		(property "Part Number" "CL05B104KO5NNNC"
 			(at 39.37 29.21 0)
 			(hide yes)
@@
 			)
 		)
-		(property "Part Number" "CL05B104KB5NNNC"
+		(property "Part Number" "CL05B104KO5NNNC"
 			(at 44.45 29.21 0)
 			(hide yes)
@@
 			)
 		)
-		(property "Value" "1k6 1%"
+		(property "Value" "1k6"
 			(at 109.728 139.954 90)
 			(show_name no)
@@
 			)
 		)
-		(property "Part Number" "RT0603BRD071K6L"
+		(property "Part Number" "RC0603FR-071K6L"
 			(at 105.41 142.24 90)
 			(hide yes)
@@
 			)
 		)
-		(property "Part Number" "CL05B104KB5NNNC"
+		(property "Part Number" "CL05B104KO5NNNC"
 			(at 54.61 46.99 0)
 			(hide yes)
@@
 			)
 		)
-		(property "Part Number" "CL05B104KB5NNNC"
+		(property "Part Number" "CL05B104KO5NNNC"
 			(at 54.61 29.21 0)
 			(hide yes)
@@
 			)
 		)
-		(property "Part Number" "CL05B104KB5NNNC"
+		(property "Part Number" "CL05B104KO5NNNC"
 			(at 228.6 39.37 0)
 			(hide yes)
@@
 			)
 		)
-		(property "Part Number" "AC0603FR-0710KL"
+		(property "Part Number" "RC0603FR-0710KL"
 			(at 81.28 77.47 0)
 			(hide yes)
@@
 			)
 		)
-		(property "Part Number" "AC0603FR-0710KL"
+		(property "Part Number" "RC0603FR-0710KL"
 			(at 38.1 101.6 0)
 			(hide yes)
@@
 			)
 		)
-		(property "Part Number" "CL05B104KB5NNNC"
+		(property "Part Number" "CL05B104KO5NNNC"
 			(at 29.21 46.99 0)
 			(hide yes)

Commit message: changes
Parts:
- C10: Part Number CL21A106KOQNNNE -> CC0805KRX5R8BB106
- C11, C12, C13, C14, C15, C16, C17, C18, C19, C20, C22, C23, C3, C4, C5, C6, C7, C8: Part Number CL05B104KO5NNNC -> CC0402KRX7R8BB104
- C21, C9: footprint Capacitor_SMD:C_0805_2012Metric -> Capacitor_SMD:C_1206_3216Metric; Part Number CL21A226MOQNNNE -> CC1206KKX5R8BB226
- C24, C25: Part Number CL05C270JB5NNNC -> CC0402JRNPO9BN270
- C26: Part Number CL05A334KQ5NNNC -> CC0402KPX5R6BB334
- R12: value 1k6 -> 1k6 1%
Changed lines of the file:
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@@
 			)
 		)
-		(property "Part Number" "CL05B104KO5NNNC"
+		(property "Part Number" "CC0402KRX7R8BB104"
 			(at 29.21 29.21 0)
 			(hide yes)
@@
 			)
 		)
-		(property "Part Number" "CL05B104KO5NNNC"
+		(property "Part Number" "CC0402KRX7R8BB104"
 			(at 39.37 46.99 0)
 			(hide yes)
@@
 			)
 		)
-		(property "Part Number" "CL05B104KO5NNNC"
+		(property "Part Number" "CC0402KRX7R8BB104"
 			(at 91.44 59.69 90)
 			(hide yes)
@@
 			)
 		)
-		(property "Part Number" "CL05C270JB5NNNC"
+		(property "Part Number" "CC0402JRNPO9BN270"
 			(at 95.25 127 90)
 			(hide yes)
@@
 			)
 		)
-		(property "Part Number" "CL05B104KO5NNNC"
+		(property "Part Number" "CC0402KRX7R8BB104"
 			(at 34.29 29.21 0)
 			(hide yes)
@@
 			)
 		)
-		(property "Part Number" "CL05B104KO5NNNC"
+		(property "Part Number" "CC0402KRX7R8BB104"
 			(at 64.77 46.99 0)
 			(hide yes)
@@
 			)
 		)
-		(property "Footprint" "Capacitor_SMD:C_0805_2012Metric"
+		(property "Footprint" "Capacitor_SMD:C_1206_3216Metric"
 			(at 64.77 29.21 0)
 			(hide yes)
@@
 			)
 		)
-		(property "Part Number" "CL21A226MOQNNNE"
+		(property "Part Number" "CC1206KKX5R8BB226"
 			(at 64.77 29.21 0)
 			(hide yes)
@@
 			)
 		)
-		(property "Part Number" "CL05B104KO5NNNC"
+		(property "Part Number" "CC0402KRX7R8BB104"
 			(at 49.53 29.21 0)
 			(hide yes)
@@
 			)
 		)
-		(property "Part Number" "CL05B104KO5NNNC"
+		(property "Part Number" "CC0402KRX7R8BB104"
 			(at 34.29 46.99 0)
 			(hide yes)
@@
 			)
 		)
-		(property "Part Number" "CL05C270JB5NNNC"
+		(property "Part Number" "CC0402JRNPO9BN270"
 			(at 95.25 134.62 90)
 			(hide yes)
@@
 			)
 		)
-		(property "Part Number" "CL05B104KO5NNNC"
+		(property "Part Number" "CC0402KRX7R8BB104"
 			(at 223.52 39.37 0)
 			(hide yes)
@@
 			)
 		)
-		(property "Footprint" "Capacitor_SMD:C_0805_2012Metric"
+		(property "Footprint" "Capacitor_SMD:C_1206_3216Metric"
 			(at 73.66 46.99 0)
 			(hide yes)
@@
 			)
 		)
-		(property "Part Number" "CL21A226MOQNNNE"
+		(property "Part Number" "CC1206KKX5R8BB226"
 			(at 73.66 46.99 0)
 			(hide yes)
@@
 			)
 		)
-		(property "Part Number" "CL05B104KO5NNNC"
+		(property "Part Number" "CC0402KRX7R8BB104"
 			(at 59.69 46.99 0)
 			(hide yes)
@@
 			)
 		)
-		(property "Part Number" "CL05B104KO5NNNC"
+		(property "Part Number" "CC0402KRX7R8BB104"
 			(at 49.53 46.99 0)
 			(hide yes)
@@
 			)
 		)
-		(property "Part Number" "CL05B104KO5NNNC"
+		(property "Part Number" "CC0402KRX7R8BB104"
 			(at 44.45 46.99 0)
 			(hide yes)
@@
 			)
 		)
-		(property "Part Number" "CL05B104KO5NNNC"
+		(property "Part Number" "CC0402KRX7R8BB104"
 			(at 91.44 62.23 90)
 			(hide yes)
@@
 			)
 		)
-		(property "Part Number" "CL21A106KOQNNNE "
+		(property "Part Number" "CC0805KRX5R8BB106"
 			(at 213.36 39.37 0)
 			(hide yes)
@@
 			)
 		)
-		(property "Part Number" "CL05B104KO5NNNC"
+		(property "Part Number" "CC0402KRX7R8BB104"
 			(at 39.37 29.21 0)
 			(hide yes)
@@
 			)
 		)
-		(property "Part Number" "CL05B104KO5NNNC"
+		(property "Part Number" "CC0402KRX7R8BB104"
 			(at 44.45 29.21 0)
 			(hide yes)
@@
 			)
 		)
-		(property "Value" "1k6"
+		(property "Value" "1k6 1%"
 			(at 109.728 139.954 90)
 			(show_name no)
@@
 			)
 		)
-		(property "Part Number" "CL05B104KO5NNNC"
+		(property "Part Number" "CC0402KRX7R8BB104"
 			(at 54.61 46.99 0)
 			(hide yes)
@@
 			)
 		)
-		(property "Part Number" "CL05B104KO5NNNC"
+		(property "Part Number" "CC0402KRX7R8BB104"
 			(at 54.61 29.21 0)
 			(hide yes)
@@
 			)
 		)
-		(property "Part Number" "CL05B104KO5NNNC"
+		(property "Part Number" "CC0402KRX7R8BB104"
 			(at 228.6 39.37 0)
 			(hide yes)
@@
 			)
 		)
-		(property "Part Number" "CL05B104KO5NNNC"
+		(property "Part Number" "CC0402KRX7R8BB104"
 			(at 29.21 46.99 0)
 			(hide yes)
@@
 			)
 		)
-		(property "Part Number" "CL05A334KQ5NNNC"
+		(property "Part Number" "CC0402KPX5R6BB334"
 			(at 81.28 142.24 0)
 			(hide yes)

Commit message: final
Parts:
- renumbered R9 to R10, R10 to R11, R11 to R12, R12 to R13, R4 to R5, R5 to R6, R6 to R7, R7 to R8, R8 to R9
Changed lines of the file:
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@@
 		(in_pos_files yes)
 		(dnp no)
-		(property "Reference" "R10"
+		(property "Reference" "R11"
 			(at 110.998 116.078 0)
 			(show_name no)
@@
 			(project "rov_usb"
 				(path "/e63e39d7-6ac0-4ffd-8aa3-1841a4541b55/49ca2e40-2d13-4810-89b0-6bfff32416b9"
-					(reference "R10")
+					(reference "R11")
 					(unit 1)
 				)
@@
 		(in_pos_files yes)
 		(dnp no)
-		(property "Reference" "R9"
+		(property "Reference" "R10"
 			(at 77.724 113.792 0)
 			(show_name no)
@@
 			(project "rov_usb"
 				(path "/e63e39d7-6ac0-4ffd-8aa3-1841a4541b55/49ca2e40-2d13-4810-89b0-6bfff32416b9"
-					(reference "R9")
+					(reference "R10")
 					(unit 1)
 				)
@@
 		(in_pos_files yes)
 		(dnp no)
-		(property "Reference" "#PWR016"
+		(property "Reference" "#PWR018"
 			(at 163.83 163.83 0)
 			(hide yes)
@@
 			(project "rov_usb"
 				(path "/e63e39d7-6ac0-4ffd-8aa3-1841a4541b55/49ca2e40-2d13-4810-89b0-6bfff32416b9"
-					(reference "#PWR016")
+					(reference "#PWR018")
 					(unit 1)
 				)
@@
 		(in_pos_files yes)
 		(dnp no)
-		(property "Reference" "#PWR013"
+		(property "Reference" "#PWR015"
 			(at 81.28 153.67 0)
 			(hide yes)
@@
 			(project "rov_usb"
 				(path "/e63e39d7-6ac0-4ffd-8aa3-1841a4541b55/49ca2e40-2d13-4810-89b0-6bfff32416b9"
-					(reference "#PWR013")
+					(reference "#PWR015")
 					(unit 1)
 				)
@@
 		(in_pos_files yes)
 		(dnp no)
-		(property "Reference" "R11"
+		(property "Reference" "R12"
 			(at 113.284 127.254 90)
 			(show_name no)
@@
 			(project "rov_usb"
 				(path "/e63e39d7-6ac0-4ffd-8aa3-1841a4541b55/49ca2e40-2d13-4810-89b0-6bfff32416b9"
-					(reference "R11")
+					(reference "R12")
 					(unit 1)
 				)
@@
 		(in_pos_files yes)
 		(dnp no)
-		(property "Reference" "R7"
+		(property "Reference" "R8"
 			(at 88.646 94.742 0)
 			(show_name no)
@@
 			(project "rov_usb"
 				(path "/e63e39d7-6ac0-4ffd-8aa3-1841a4541b55/49ca2e40-2d13-4810-89b0-6bfff32416b9"
-					(reference "R7")
+					(reference "R8")
 					(unit 1)
 				)
@@
 		(in_pos_files yes)
 		(dnp no)
-		(property "Reference" "#PWR03"
+		(property "Reference" "#PWR05"
 			(at 64.77 40.64 0)
 			(hide yes)
@@
 			(project "rov_usb"
 				(path "/e63e39d7-6ac0-4ffd-8aa3-1841a4541b55/49ca2e40-2d13-4810-89b0-6bfff32416b9"
-					(reference "#PWR03")
+					(reference "#PWR05")
 					(unit 1)
 				)
@@
 		(in_pos_files yes)
 		(dnp no)
-		(property "Reference" "#PWR010"
+		(property "Reference" "#PWR012"
 			(at 107.95 116.84 0)
 			(hide yes)
@@
 			(project "rov_usb"
 				(path "/e63e39d7-6ac0-4ffd-8aa3-1841a4541b55/49ca2e40-2d13-4810-89b0-6bfff32416b9"
-					(reference "#PWR010")
+					(reference "#PWR012")
 					(unit 1)
 				)
@@
 		(in_pos_files yes)
 		(dnp no)
-		(property "Reference" "#PWR012"
+		(property "Reference" "#PWR014"
 			(at 86.36 138.43 0)
 			(hide yes)
@@
 			(project "rov_usb"
 				(path "/e63e39d7-6ac0-4ffd-8aa3-1841a4541b55/49ca2e40-2d13-4810-89b0-6bfff32416b9"
-					(reference "#PWR012")
+					(reference "#PWR014")
 					(unit 1)
 				)
@@
 		(in_pos_files yes)
 		(dnp no)
-		(property "Reference" "#PWR04"
+		(property "Reference" "#PWR06"
 			(at 135.89 45.72 0)
 			(hide yes)
@@
 			(project "rov_usb"
 				(path "/e63e39d7-6ac0-4ffd-8aa3-1841a4541b55/49ca2e40-2d13-4810-89b0-6bfff32416b9"
-					(reference "#PWR04")
+					(reference "#PWR06")
 					(unit 1)
 				)
@@
 		(in_pos_files yes)
 		(dnp no)
-		(property "Reference" "R6"
+		(property "Reference" "R7"
 			(at 81.026 94.742 0)
 			(show_name no)
@@
 			(project "rov_usb"
 				(path "/e63e39d7-6ac0-4ffd-8aa3-1841a4541b55/49ca2e40-2d13-4810-89b0-6bfff32416b9"
-					(reference "R6")
+					(reference "R7")
 					(unit 1)
 				)
@@
 		(in_pos_files yes)
 		(dnp no)
-		(property "Reference" "#PWR06"
+		(property "Reference" "#PWR08"
 			(at 213.36 50.8 0)
 			(hide yes)
@@
 			(project "rov_usb"
 				(path "/e63e39d7-6ac0-4ffd-8aa3-1841a4541b55/49ca2e40-2d13-4810-89b0-6bfff32416b9"
-					(reference "#PWR06")
+					(reference "#PWR08")
 					(unit 1)
 				)
@@
 		(in_pos_files yes)
 		(dnp no)
-		(property "Reference" "#PWR05"
+		(property "Reference" "#PWR07"
 			(at 163.83 46.99 0)
 			(hide yes)
@@
 			(project "rov_usb"
 				(path "/e63e39d7-6ac0-4ffd-8aa3-1841a4541b55/49ca2e40-2d13-4810-89b0-6bfff32416b9"
-					(reference "#PWR05")
+					(reference "#PWR07")
 					(unit 1)
 				)
@@
 		(in_pos_files yes)
 		(dnp no)
-		(property "Reference" "R5"
+		(property "Reference" "R6"
 			(at 70.104 94.742 0)
 			(show_name no)
@@
 			(project "rov_usb"
 				(path "/e63e39d7-6ac0-4ffd-8aa3-1841a4541b55/49ca2e40-2d13-4810-89b0-6bfff32416b9"
-					(reference "R5")
+					(reference "R6")
 					(unit 1)
 				)
@@
 		(in_pos_files yes)
 		(dnp no)
-		(property "Reference" "#PWR011"
+		(property "Reference" "#PWR013"
 			(at 55.88 129.54 0)
 			(hide yes)
@@
 			(project "rov_usb"
 				(path "/e63e39d7-6ac0-4ffd-8aa3-1841a4541b55/49ca2e40-2d13-4810-89b0-6bfff32416b9"
-					(reference "#PWR011")
+					(reference "#PWR013")
 					(unit 1)
 				)
@@
 		(in_pos_files yes)
 		(dnp no)
-		(property "Reference" "#PWR09"
+		(property "Reference" "#PWR011"
 			(at 55.88 93.98 0)
 			(hide yes)
@@
 			(project "rov_usb"
 				(path "/e63e39d7-6ac0-4ffd-8aa3-1841a4541b55/49ca2e40-2d13-4810-89b0-6bfff32416b9"
-					(reference "#PWR09")
+					(reference "#PWR011")
 					(unit 1)
 				)
@@
 		(in_pos_files yes)
 		(dnp no)
-		(property "Reference" "R12"
+		(property "Reference" "R13"
 			(at 102.616 139.954 90)
 			(show_name no)
@@
 			(project "rov_usb"
 				(path "/e63e39d7-6ac0-4ffd-8aa3-1841a4541b55/49ca2e40-2d13-4810-89b0-6bfff32416b9"
-					(reference "R12")
+					(reference "R13")
 					(unit 1)
 				)
@@
 		(in_pos_files yes)
 		(dnp no)
-		(property "Reference" "#PWR07"
+		(property "Reference" "#PWR09"
 			(at 73.66 58.42 0)
 			(hide yes)
@@
 			(project "rov_usb"
 				(path "/e63e39d7-6ac0-4ffd-8aa3-1841a4541b55/49ca2e40-2d13-4810-89b0-6bfff32416b9"
-					(reference "#PWR07")
+					(reference "#PWR09")
 					(unit 1)
 				)
@@
 		(in_pos_files yes)
 		(dnp no)
-		(property "Reference" "#PWR015"
+		(property "Reference" "#PWR017"
 			(at 212.09 154.94 0)
 			(hide yes)
@@
 			(project "rov_usb"
 				(path "/e63e39d7-6ac0-4ffd-8aa3-1841a4541b55/49ca2e40-2d13-4810-89b0-6bfff32416b9"
-					(reference "#PWR015")
+					(reference "#PWR017")
 					(unit 1)
 				)
@@
 		(in_pos_files yes)
 		(dnp no)
-		(property "Reference" "#PWR014"
+		(property "Reference" "#PWR016"
 			(at 115.57 153.67 0)
 			(hide yes)
@@
 			(project "rov_usb"
 				(path "/e63e39d7-6ac0-4ffd-8aa3-1841a4541b55/49ca2e40-2d13-4810-89b0-6bfff32416b9"
-					(reference "#PWR014")
+					(reference "#PWR016")
 					(unit 1)
 				)
@@
 		(in_pos_files yes)
 		(dnp no)
-		(property "Reference" "R4"
+		(property "Reference" "R5"
 			(at 77.724 75.692 0)
 			(show_name no)
@@
 			(project "rov_usb"
 				(path "/e63e39d7-6ac0-4ffd-8aa3-1841a4541b55/49ca2e40-2d13-4810-89b0-6bfff32416b9"
-					(reference "R4")
+					(reference "R5")
 					(unit 1)
 				)
@@
 		(in_pos_files yes)
 		(dnp no)
-		(property "Reference" "R8"
+		(property "Reference" "R9"
 			(at 41.656 99.822 0)
 			(show_name no)
@@
 			(project "rov_usb"
 				(path "/e63e39d7-6ac0-4ffd-8aa3-1841a4541b55/49ca2e40-2d13-4810-89b0-6bfff32416b9"
-					(reference "R8")
+					(reference "R9")
 					(unit 1)
 				)
@@
 		(in_pos_files yes)
 		(dnp no)
-		(property "Reference" "#PWR08"
+		(property "Reference" "#PWR010"
 			(at 81.28 76.2 0)
 			(hide yes)
@@
 			(project "rov_usb"
 				(path "/e63e39d7-6ac0-4ffd-8aa3-1841a4541b55/49ca2e40-2d13-4810-89b0-6bfff32416b9"
-					(reference "#PWR08")
+					(reference "#PWR010")
 					(unit 1)
 				)

Commit message: move parts to project specific libs
Parts:
- removed U1: UPD720201K8-701-BAC-A, snadol:QFN68_8X8_REN, symbol snadol:UPD720201K8-7x1-BAC-A
- removed U2: SST25VF512A-33-4C-SAE, snadol:SST25VF512A, symbol snadol:SST25VF512A-33-4C-SAE
- added U1: UPD720201K8-7x1-BAC-A, ROV_PCIe_USB_HUB:QFN-68-1EP_8x8mm_P0.4mm_EP6.2x6.2mm, symbol ROV_PCIe_USB_HUB:UPD720201K8-7x1-BAC-A
- added U2: SST25VF512A-33-4C-SAE, Package_SO:SOIC-8_3.9x4.9mm_P1.27mm, symbol ROV_PCIe_USB_HUB:SST25VF512A-33-4C-SAE
Connections:
- net +1.05V: now also U1.12 (VDD10), U1.28 (VDD10), U1.37 (VDD10), U1.43 (VDD10), U1.46 (VDD10), U1.54 (VDD10), U1.60 (VDD10), U1.63 (VDD10), U1.9 (VDD10)
- net +3.3V: now also U1.15 (VDD33), U1.29 (VDD33), U1.40 (VDD33), U1.49 (VDD33), U1.57 (VDD33), U1.66 (VDD33), U2.7 (*HOLD), U2.8 (VDD)
- net +3.3V_A: now also U1.32 (AVDD33), U1.6 (AVDD33)
- net 1V05_PG: now also U1.14 (PONRSTB)
- net GND: now also U1.34 (IC(L)), U1.38 (U3RXDP1), U1.39 (U3RXDN1), U1.47 (U3RXDP2), U1.48 (U3RXDN2), U1.55 (U3RXDP3), U1.56 (U3RXDN3), U1.69 (GND), U2.4 (VSS)
- net PCIE_CLKREQ_N: now also U1.13 (PECREQB)
- net PCIE_DET_WAKE: now also U1.3 (PEWAKEB)
- net PCIE_RST_B: now also U1.2 (PERSTB)
- net PI_PCIE_CLK_N: now also U1.5 (PECLKN)
- net PI_PCIE_CLK_P: now also U1.4 (PECLKP)
- net PI_PCIE_TX_N: now also U1.11 (PERXN)
- net PI_PCIE_TX_P: now also U1.10 (PERXP)
- net UPD_PCIE_TX_N: now also U1.8 (PETXN)
- net UPD_PCIE_TX_P: now also U1.7 (PETXP)
- net USB1_DN: now also U1.42 (U2DM1)
- net USB1_DP: now also U1.41 (U2DP1)
- net USB2_DN: now also U1.51 (U2DM2)
- net USB2_DP: now also U1.50 (U2DP2)
- net USB3_DN: now also U1.59 (U2DM3)
- net USB3_DP: now also U1.58 (U2DP3)
- net USB4_DN: now also U1.68 (U2DM4)
- net USB4_DP: now also U1.67 (U2DP4)
- net USB4_SSRXN: now also U1.65 (U3RXDN4)
- net USB4_SSRXP: now also U1.64 (U3RXDP4)
- net USB4_SSTXN: now also U1.62 (U3TXDN4)
- net USB4_SSTXP: now also U1.61 (U3TXDP4)
- net at R11.2: now also U1.20 (OCI4B), U1.22 (OCI3B), U1.24 (OCI2B), U1.26 (OCI1B)
- net at R10.1: now also U1.18 (SPISCK), U2.6 (SCK)
- net at R12.2: now also U1.30 (XT2)
- net at R8.2: now also U1.17 (SPICSB), U2.1 (*CE)
- net at C25.2, Y1.3: now also U1.31 (XT1)
- net at R7.2: now also U1.19 (SPISI), U2.5 (SI)
- net at R6.2: now also U1.16 (SPISO), U2.2 (SO)
- net at R13.2: now also U1.33 (RREF)
- net at R9.2: now also U2.3 (*WP)
