File: ROV_PCIe_USB_HUB_FINAL/Power.kicad_sch (KiCad schematic)
At the start: 18 parts, among them U15 TPS62A02APDDC, U16 TPS62A02APDDC

Commit message: changes
Parts:
- L1, L2: value BDCC00201208R47MWA -> 1u; footprint Inductor_SMD:L_0805_2012Metric -> Inductor_SMD:L_1008_2520Metric; Part Number BDCC00201208R47MWA -> DFE252012F-1R0M
- renumbered C59 to C67, C60 to C68, C61 to C69, C62 to C70, C63 to C71, C64 to C72, C65 to C73, C66 to C74, R16 to R43, R21 to R44, R26 to R45, R31 to R46, R34 to R47, R35 to R48
Other:
- note removed: "470nH Isat >= 3A DCR < 40mOhm"

Commit message: work
Parts:
- renumbered C67 to C66, C68 to C67, C69 to C68, C70 to C69, C71 to C70, C72 to C71, C73 to C72, C74 to C73, R43 to R39, R44 to R40, R45 to R41, R46 to R42, R47 to R43, R48 to R44
Changed lines of the file:
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@@
 		(dnp yes)
 		(fields_autoplaced yes)
-		(property "Reference" "C71"
+		(property "Reference" "C70"
 			(at 138.43 62.2362 0)
 			(show_name no)
@@
 			(project "ROV_PCIE_USB_HUB_FINAL"
 				(path "/95e7ccb6-701a-4570-b93f-f5431fbf25de/42000762-0d3e-4a2e-8bb0-02360d8a7156"
-					(reference "C71")
+					(reference "C70")
 					(unit 1)
 				)
@@
 		(in_pos_files yes)
 		(dnp no)
-		(property "Reference" "R44"
+		(property "Reference" "R40"
 			(at 106.68 102.8699 0)
 			(show_name no)
@@
 			(project "ROV_PCIE_USB_HUB_FINAL"
 				(path "/95e7ccb6-701a-4570-b93f-f5431fbf25de/42000762-0d3e-4a2e-8bb0-02360d8a7156"
-					(reference "R44")
+					(reference "R40")
 					(unit 1)
 				)
@@
 		(dnp yes)
 		(fields_autoplaced yes)
-		(property "Reference" "C72"
+		(property "Reference" "C71"
 			(at 138.43 114.3062 0)
 			(show_name no)
@@
 			(project "ROV_PCIE_USB_HUB_FINAL"
 				(path "/95e7ccb6-701a-4570-b93f-f5431fbf25de/42000762-0d3e-4a2e-8bb0-02360d8a7156"
-					(reference "C72")
+					(reference "C71")
 					(unit 1)
 				)
@@
 		(in_pos_files yes)
 		(dnp no)
-		(property "Reference" "C68"
+		(property "Reference" "C67"
 			(at 72.39 120.6562 0)
 			(show_name no)
@@
 			(project "ROV_PCIE_USB_HUB_FINAL"
 				(path "/95e7ccb6-701a-4570-b93f-f5431fbf25de/42000762-0d3e-4a2e-8bb0-02360d8a7156"
-					(reference "C68")
+					(reference "C67")
 					(unit 1)
 				)
@@
 		(dnp no)
 		(fields_autoplaced yes)
-		(property "Reference" "C74"
+		(property "Reference" "C73"
 			(at 151.13 118.1162 0)
 			(show_name no)
@@
 			(project "ROV_PCIE_USB_HUB_FINAL"
 				(path "/95e7ccb6-701a-4570-b93f-f5431fbf25de/42000762-0d3e-4a2e-8bb0-02360d8a7156"
-					(reference "C74")
+					(reference "C73")
 					(unit 1)
 				)
@@
 		(in_pos_files yes)
 		(dnp no)
-		(property "Reference" "C69"
+		(property "Reference" "C68"
 			(at 82.55 68.5862 0)
 			(show_name no)
@@
 			(project "ROV_PCIE_USB_HUB_FINAL"
 				(path "/95e7ccb6-701a-4570-b93f-f5431fbf25de/42000762-0d3e-4a2e-8bb0-02360d8a7156"
-					(reference "C69")
+					(reference "C68")
 					(unit 1)
 				)
@@
 		(in_pos_files yes)
 		(dnp no)
-		(property "Reference" "C70"
+		(property "Reference" "C69"
 			(at 82.55 120.6562 0)
 			(show_name no)
@@
 			(project "ROV_PCIE_USB_HUB_FINAL"
 				(path "/95e7ccb6-701a-4570-b93f-f5431fbf25de/42000762-0d3e-4a2e-8bb0-02360d8a7156"
-					(reference "C70")
+					(reference "C69")
 					(unit 1)
 				)
@@
 		(in_pos_files yes)
 		(dnp no)
-		(property "Reference" "R43"
+		(property "Reference" "R39"
 			(at 106.68 48.2599 0)
 			(show_name no)
@@
 			(project "ROV_PCIE_USB_HUB_FINAL"
 				(path "/95e7ccb6-701a-4570-b93f-f5431fbf25de/42000762-0d3e-4a2e-8bb0-02360d8a7156"
-					(reference "R43")
+					(reference "R39")
 					(unit 1)
 				)
@@
 		(dnp no)
 		(fields_autoplaced yes)
-		(property "Reference" "R46"
+		(property "Reference" "R42"
 			(at 127 69.8499 0)
 			(show_name no)
@@
 			(project "ROV_PCIE_USB_HUB_FINAL"
 				(path "/95e7ccb6-701a-4570-b93f-f5431fbf25de/42000762-0d3e-4a2e-8bb0-02360d8a7156"
-					(reference "R46")
+					(reference "R42")
 					(unit 1)
 				)
@@
 		(dnp no)
 		(fields_autoplaced yes)
-		(property "Reference" "C73"
+		(property "Reference" "C72"
 			(at 151.13 66.0462 0)
 			(show_name no)
@@
 			(project "ROV_PCIE_USB_HUB_FINAL"
 				(path "/95e7ccb6-701a-4570-b93f-f5431fbf25de/42000762-0d3e-4a2e-8bb0-02360d8a7156"
-					(reference "C73")
+					(reference "C72")
 					(unit 1)
 				)
@@
 		(in_pos_files yes)
 		(dnp no)
-		(property "Reference" "C67"
+		(property "Reference" "C66"
 			(at 72.39 68.5862 0)
 			(show_name no)
@@
 			(project "ROV_PCIE_USB_HUB_FINAL"
 				(path "/95e7ccb6-701a-4570-b93f-f5431fbf25de/42000762-0d3e-4a2e-8bb0-02360d8a7156"
-					(reference "C67")
+					(reference "C66")
 					(unit 1)
 				)
@@
 		(dnp no)
 		(fields_autoplaced yes)
-		(property "Reference" "R47"
+		(property "Reference" "R43"
 			(at 127 114.2999 0)
 			(show_name no)
@@
 			(project "ROV_PCIE_USB_HUB_FINAL"
 				(path "/95e7ccb6-701a-4570-b93f-f5431fbf25de/42000762-0d3e-4a2e-8bb0-02360d8a7156"
-					(reference "R47")
+					(reference "R43")
 					(unit 1)
 				)
@@
 		(dnp no)
 		(fields_autoplaced yes)
-		(property "Reference" "R45"
+		(property "Reference" "R41"
 			(at 127 62.2299 0)
 			(show_name no)
@@
 			(project "ROV_PCIE_USB_HUB_FINAL"
 				(path "/95e7ccb6-701a-4570-b93f-f5431fbf25de/42000762-0d3e-4a2e-8bb0-02360d8a7156"
-					(reference "R45")
+					(reference "R41")
 					(unit 1)
 				)
@@
 		(dnp no)
 		(fields_autoplaced yes)
-		(property "Reference" "R48"
+		(property "Reference" "R44"
 			(at 127 121.9199 0)
 			(show_name no)
@@
 			(project "ROV_PCIE_USB_HUB_FINAL"
 				(path "/95e7ccb6-701a-4570-b93f-f5431fbf25de/42000762-0d3e-4a2e-8bb0-02360d8a7156"
-					(reference "R48")
+					(reference "R44")
 					(unit 1)
 				)
@@
 		(dnp no)
 		(fields_autoplaced yes)
-		(property "Reference" "#FLG08"
+		(property "Reference" "#FLG04"
 			(at 146.05 109.855 0)
 			(hide yes)
@@
 			(project "ROV_PCIE_USB_HUB_FINAL"
 				(path "/95e7ccb6-701a-4570-b93f-f5431fbf25de/42000762-0d3e-4a2e-8bb0-02360d8a7156"
-					(reference "#FLG08")
+					(reference "#FLG04")
 					(unit 1)
 				)
@@
 		(dnp no)
 		(fields_autoplaced yes)
-		(property "Reference" "#FLG07"
+		(property "Reference" "#FLG03"
 			(at 146.05 57.785 0)
 			(hide yes)
@@
 			(project "ROV_PCIE_USB_HUB_FINAL"
 				(path "/95e7ccb6-701a-4570-b93f-f5431fbf25de/42000762-0d3e-4a2e-8bb0-02360d8a7156"
-					(reference "#FLG07")
+					(reference "#FLG03")
 					(unit 1)
 				)
