File: ROV_PCIe_USB_HUB_FINAL/Hub1.kicad_sch (KiCad schematic)
At the start: 21 parts, among them J2 SM04B-SRSS-TB, J3 SM04B-SRSS-TB, U3 USB2422/MJ, U4 TPS2051CDBV, U5 TPS2051CDBV, Y2 ABM8-24.000MHZ-B2-T

Commit message: changes
Parts:
- removed FB2: 220 Ohm @ 100MHz, low DCR, Inductor_SMD:L_0805_2012Metric, symbol Device:FerriteBead_Small
- added C35, C36: 10u, Capacitor_SMD:C_0805_2012Metric, symbol Device:C_Small
- added R18: 100k, Resistor_SMD:R_0603_1608Metric, symbol Device:R_Small_US
- U3: footprint Package_DFN_QFN:VQFN-24-1EP_4x4mm_P0.5mm_EP2.5x2.5mm_ThermalVias -> ROV_PCIe_USB_HUB:QFN-24-1EP_4x4mm_P0.5mm_EP2.5x2.5mm_ThermalVias
- Y2: value ABM8-24.000MHZ-B2-T -> ABM11-24.000MHZ-D2X-T; footprint Crystal:Crystal_SMD_3225-4Pin_3.2x2.5mm -> Crystal:Crystal_SMD_2016-4Pin_2.0x1.6mm
- renumbered C26 to C27, C27 to C28, C28 to C29, C29 to C30, C30 to C31, C31 to C32, C32 to C33, C33 to C34, J2 to J4, J3 to J5, R13 to R15, R14 to R16, R15 to R17, R17 to R19, R36 to R20, R40 to R21
Connections:
- net +3.3V: now also C29.1, C32.1, C33.1, C34.1, U3.1 (VDD33), U3.16 (VBUS_DET), U3.18 (VDD33), U3.9 (VDD33)
- net GND: now also C35.2, C36.2, R18.2; no longer U3.14 (SMBCLK/CFG_SEL0)
- net VBUS: no longer U3.16 (VBUS_DET)
- net at J4.1 (Pin_1), U4.1 (OUT): now also C35.1
- net at J5.1 (Pin_1), U5.1 (OUT): now also C36.1
- new net: R18.1, U3.14 (SMBCLK/CFG_SEL0)
Other:
- note removed: "BLM21PG221SN1D"

Commit message: work
Parts:
- removed R16: 0, Resistor_SMD:R_0402_1005Metric, symbol Device:R_Small_US
- C26: renamed from C27; value 27p -> 10p
- C27: renamed from C28; value 27p -> 10p
- Y2: value ABM11-24.000MHZ-D2X-T -> ECS-240-8-37B-CKY-TR
- renumbered C29 to C28, C30 to C29, C31 to C30, C32 to C31, C33 to C32, C34 to C33, C35 to C34, C36 to C35, R17 to R16, R18 to R17, R19 to R18, R20 to R19, R21 to R20
Connections:
- net at C26.2, Y2.1: now also U3.22 (XTALIN/CLKIN)
Other:
- moved on the sheet: C34, C35, J4, J5, R19, R20, U4, U5

Commit message: changes
Other:
- moved on the sheet: C26, C27, C28, C29, C30, C31, C33, C34, C35, J4, J5, R15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
