File: ROV_PCIe_USB_HUB_FINAL/ROV_PCIE_USB_HUB_FINAL.kicad_pcb (KiCad board)
At the start: 2 copper layers, 65 x 56.5 mm, 13 parts, among them J1 USB_A_Stacked, J2 USB_A_Stacked, J3 USB_A_Stacked, J4 USB_A_Stacked, U1 UPD720202K8-7x1-BAA, U2 USB2514B_Bi, U3 USB2514B_Bi, U4 USB2514B_Bi, U5 USB2514B_Bi

Commit message: work
Parts:
- added C1: 100n, Capacitor_SMD:C_0402_1005Metric, F.Cu at (131.0, 48.8)
- added C10: 100n, Capacitor_SMD:C_0402_1005Metric, F.Cu at (133.9, 54.7)
- added C11: 100n, Capacitor_SMD:C_0402_1005Metric, F.Cu at (133.9, 56.7)
- added C12: 100n, Capacitor_SMD:C_0402_1005Metric, F.Cu at (133.9, 58.7)
- added C13: 100n, Capacitor_SMD:C_0402_1005Metric, F.Cu at (136.8, 48.8)
- added C14: 100n, Capacitor_SMD:C_0402_1005Metric, F.Cu at (136.8, 50.8)
- added C15: 100n, Capacitor_SMD:C_0402_1005Metric, F.Cu at (136.8, 52.7)
- added C16: 22u, Capacitor_SMD:C_1206_3216Metric, F.Cu at (143.0, 61.3)
- added C17: 100n, Capacitor_SMD:C_0402_1005Metric, F.Cu at (136.8, 54.7)
- added C18: 22u, Capacitor_SMD:C_1206_3216Metric, F.Cu at (143.0, 64.7)
- added C19: 100n, Capacitor_SMD:C_0402_1005Metric, F.Cu at (136.8, 56.7)
- added C2: 100n, Capacitor_SMD:C_0402_1005Metric, F.Cu at (131.0, 50.8)
- added C20: 100n, Capacitor_SMD:C_0402_1005Metric, F.Cu at (136.8, 58.7)
- added C21: 27p, Capacitor_SMD:C_0402_1005Metric, F.Cu at (139.6, 48.8)
- added C22: 27p, Capacitor_SMD:C_0402_1005Metric, F.Cu at (139.6, 50.8)
- added C23: 10u, Capacitor_SMD:C_0805_2012Metric, F.Cu at (147.3, 56.6)
- added C24: 100n, Capacitor_SMD:C_0402_1005Metric, F.Cu at (139.6, 52.7)
- added C25: 100n, Capacitor_SMD:C_0402_1005Metric, F.Cu at (139.6, 54.7)
- added C26: 27p, Capacitor_SMD:C_0402_1005Metric, F.Cu at (137.0, 94.8)
- added C27: 27p, Capacitor_SMD:C_0402_1005Metric, F.Cu at (137.0, 96.7)
- added C28: 100n, Capacitor_SMD:C_0402_1005Metric, F.Cu at (137.0, 98.7)
- added C29: 100n, Capacitor_SMD:C_0402_1005Metric, F.Cu at (137.0, 100.7)
- added C3: 100n, Capacitor_SMD:C_0402_1005Metric, F.Cu at (131.0, 52.7)
- added C30: 1u, Capacitor_SMD:C_0603_1608Metric, F.Cu at (140.4, 95.0)
- added C31: 100n, Capacitor_SMD:C_0402_1005Metric, F.Cu at (137.0, 102.6)
- added C32: 100n, Capacitor_SMD:C_0402_1005Metric, F.Cu at (137.0, 104.6)
- added C33: 10u, Capacitor_SMD:C_0805_2012Metric, F.Cu at (145.2, 111.6)
- added C34: 27p, Capacitor_SMD:C_0402_1005Metric, F.Cu at (159.9, 73.0)
- added C35: 27p, Capacitor_SMD:C_0402_1005Metric, F.Cu at (159.9, 75.0)
- added C36: 100n, Capacitor_SMD:C_0402_1005Metric, F.Cu at (159.9, 76.9)
- added C37: 100n, Capacitor_SMD:C_0402_1005Metric, F.Cu at (159.9, 78.9)
- added C38: 1u, Capacitor_SMD:C_0603_1608Metric, F.Cu at (163.3, 73.3)
- added C39: 100n, Capacitor_SMD:C_0402_1005Metric, F.Cu at (159.9, 80.9)
- added C4: 100n, Capacitor_SMD:C_0402_1005Metric, F.Cu at (131.0, 54.7)
- added C40: 100n, Capacitor_SMD:C_0402_1005Metric, F.Cu at (159.9, 82.8)
- added C41: 10u, Capacitor_SMD:C_0805_2012Metric, F.Cu at (168.1, 89.9)
- added C42: 27p, Capacitor_SMD:C_0402_1005Metric, F.Cu at (137.0, 73.0)
- added C43: 27p, Capacitor_SMD:C_0402_1005Metric, F.Cu at (137.0, 75.0)
- added C44: 100n, Capacitor_SMD:C_0402_1005Metric, F.Cu at (137.0, 76.9)
- added C45: 100n, Capacitor_SMD:C_0402_1005Metric, F.Cu at (137.0, 78.9)
- added C46: 1u, Capacitor_SMD:C_0603_1608Metric, F.Cu at (140.4, 73.3)
- added C47: 100n, Capacitor_SMD:C_0402_1005Metric, F.Cu at (137.0, 80.9)
- added C48: 100n, Capacitor_SMD:C_0402_1005Metric, F.Cu at (137.0, 82.8)
- added C49: 10u, Capacitor_SMD:C_0805_2012Metric, F.Cu at (145.2, 89.9)
- added C5: 100n, Capacitor_SMD:C_0402_1005Metric, F.Cu at (131.0, 56.7)
- added C50: 27p, Capacitor_SMD:C_0402_1005Metric, F.Cu at (161.9, 48.8)
- added C51: 27p, Capacitor_SMD:C_0402_1005Metric, F.Cu at (161.9, 50.8)
- added C52: 100n, Capacitor_SMD:C_0402_1005Metric, F.Cu at (161.9, 52.7)
- added C53: 100n, Capacitor_SMD:C_0402_1005Metric, F.Cu at (161.9, 54.7)
- added C54: 1u, Capacitor_SMD:C_0603_1608Metric, F.Cu at (165.4, 49.1)
- added C55: 100n, Capacitor_SMD:C_0402_1005Metric, F.Cu at (161.9, 56.7)
- added C56: 100n, Capacitor_SMD:C_0402_1005Metric, F.Cu at (161.9, 58.7)
- added C57: 10u, Capacitor_SMD:C_0805_2012Metric, F.Cu at (170.1, 65.7)
- added C58: 330n, Capacitor_SMD:C_0402_1005Metric, F.Cu at (173.5, 98.1)
- added C59: 10u, Capacitor_SMD:C_0805_2012Metric, F.Cu at (163.8, 95.3)
- added C6: 100n, Capacitor_SMD:C_0402_1005Metric, F.Cu at (131.0, 58.7)
- added C60: 10u, Capacitor_SMD:C_0805_2012Metric, F.Cu at (163.8, 98.3)
- added C61: 100n, Capacitor_SMD:C_0402_1005Metric, F.Cu at (160.2, 94.8)
- added C62: 100n, Capacitor_SMD:C_0402_1005Metric, F.Cu at (160.2, 96.7)
- added C63: 10p, Capacitor_SMD:C_0402_1005Metric, F.Cu at (160.2, 98.7)
- added C64: 22p, Capacitor_SMD:C_0402_1005Metric, F.Cu at (160.2, 100.7)
- added C65: 22u, Capacitor_SMD:C_1206_3216Metric, F.Cu at (161.6, 103.3)
- added C66: 22u, Capacitor_SMD:C_1206_3216Metric, F.Cu at (161.6, 106.7)
- added C7: 100n, Capacitor_SMD:C_0402_1005Metric, F.Cu at (133.9, 48.8)
- added C8: 100n, Capacitor_SMD:C_0402_1005Metric, F.Cu at (133.9, 50.8)
- added C9: 100n, Capacitor_SMD:C_0402_1005Metric, F.Cu at (133.9, 52.7)
- added D1: BAT54W, Package_TO_SOT_SMD:SOT-323_SC-70, F.Cu at (174.0, 95.5)
- added FB1: 220 Ohm @ 100MHz, low DCR, Inductor_SMD:L_0805_2012Metric, F.Cu at (147.4, 53.7)
- added FB2: 220 Ohm @ 100MHz, low DCR, Inductor_SMD:L_0805_2012Metric, F.Cu at (140.7, 111.5)
- added FB3: 220 Ohm @ 100MHz, low DCR, Inductor_SMD:L_0805_2012Metric, F.Cu at (163.6, 89.7)
- added FB4: 220 Ohm @ 100MHz, low DCR, Inductor_SMD:L_0805_2012Metric, F.Cu at (140.7, 89.7)
- added FB5: 220 Ohm @ 100MHz, low DCR, Inductor_SMD:L_0805_2012Metric, F.Cu at (165.6, 65.5)
- added J5: SM04B-SRSS-TB, Connector_JST:JST_SH_SM04B-SRSS-TB_1x04-1MP_P1.00mm_Horizontal, F.Cu at (154.0, 83.4)
- added J6: SM04B-SRSS-TB, Connector_JST:JST_SH_SM04B-SRSS-TB_1x04-1MP_P1.00mm_Horizontal, F.Cu at (131.1, 75.8)
- added J7: SM04B-SRSS-TB, Connector_JST:JST_SH_SM04B-SRSS-TB_1x04-1MP_P1.00mm_Horizontal, F.Cu at (131.1, 83.4)
- added J8: SM04B-SRSS-TB, Connector_JST:JST_SH_SM04B-SRSS-TB_1x04-1MP_P1.00mm_Horizontal, F.Cu at (156.1, 51.6)
- added J9: SM04B-SRSS-TB, Connector_JST:JST_SH_SM04B-SRSS-TB_1x04-1MP_P1.00mm_Horizontal, F.Cu at (156.1, 59.2)
- added L1: BDCC00201208R47MWA, Inductor_SMD:L_0805_2012Metric, F.Cu at (155.9, 104.4)
- added L2: BDCC00201208R47MWA, Inductor_SMD:L_0805_2012Metric, F.Cu at (155.9, 107.1)
- added R1: 100k, Resistor_SMD:R_0603_1608Metric, F.Cu at (170.1, 95.0)
- added R10: 1k6 1%, Resistor_SMD:R_0603_1608Metric, F.Cu at (143.1, 56.1)
- added R11: 10k, Resistor_SMD:R_0402_1005Metric, F.Cu at (128.1, 58.8)
- added R12: 0, Resistor_SMD:R_0402_1005Metric, F.Cu at (128.1, 60.8)
- added R13: 12k, Resistor_SMD:R_0603_1608Metric, F.Cu at (140.4, 97.5)
- added R14: 0, Resistor_SMD:R_0402_1005Metric, F.Cu at (133.4, 110.0)
- added R15: 100k, Resistor_SMD:R_0603_1608Metric, F.Cu at (140.4, 100.0)
- added R16: 10k, Resistor_SMD:R_0603_1608Metric, F.Cu at (151.6, 95.0)
- added R17: 100k, Resistor_SMD:R_0603_1608Metric, F.Cu at (140.4, 102.6)
- added R18: 12k, Resistor_SMD:R_0603_1608Metric, F.Cu at (163.3, 75.8)
- added R19: 0, Resistor_SMD:R_0402_1005Metric, F.Cu at (156.3, 88.2)
- added R2: 5k1, Resistor_SMD:R_0603_1608Metric, F.Cu at (170.1, 97.5)
- added R20: 100k, Resistor_SMD:R_0603_1608Metric, F.Cu at (163.3, 78.3)
- added R21: 10k, Resistor_SMD:R_0603_1608Metric, F.Cu at (151.6, 97.5)
- added R22: 100k, Resistor_SMD:R_0603_1608Metric, F.Cu at (163.3, 80.8)
- added R23: 12k, Resistor_SMD:R_0603_1608Metric, F.Cu at (140.4, 75.8)
- added R24: 0, Resistor_SMD:R_0402_1005Metric, F.Cu at (133.4, 88.2)
- added R25: 100k, Resistor_SMD:R_0603_1608Metric, F.Cu at (140.4, 78.3)
- added R26: 453k, Resistor_SMD:R_0603_1608Metric, F.Cu at (151.6, 100.0)
- added R27: 100k, Resistor_SMD:R_0603_1608Metric, F.Cu at (140.4, 80.8)
- added R28: 12k, Resistor_SMD:R_0603_1608Metric, F.Cu at (165.4, 51.6)
- added R29: 0, Resistor_SMD:R_0402_1005Metric, F.Cu at (158.3, 64.0)
- added R3: 10k, Resistor_SMD:R_0603_1608Metric, F.Cu at (170.1, 100.0)
- added R30: 100k, Resistor_SMD:R_0603_1608Metric, F.Cu at (165.4, 54.1)
- added R31: 100k, Resistor_SMD:R_0603_1608Metric, F.Cu at (151.6, 102.6)
- added R32: 100k, Resistor_SMD:R_0603_1608Metric, F.Cu at (165.4, 56.6)
- added R33: 10k, Resistor_SMD:R_0603_1608Metric, F.Cu at (170.1, 102.6)
- added R34: 75k, Resistor_SMD:R_0603_1608Metric, F.Cu at (151.6, 105.1)
- added R35: 100k, Resistor_SMD:R_0603_1608Metric, F.Cu at (151.6, 107.6)
- added R4: 10k, Resistor_SMD:R_0402_1005Metric, F.Cu at (128.1, 48.8)
- added R5: 10k, Resistor_SMD:R_0402_1005Metric, F.Cu at (128.1, 50.8)
- added R6: 10k, Resistor_SMD:R_0402_1005Metric, F.Cu at (128.1, 52.8)
- added R7: 100k, Resistor_SMD:R_0603_1608Metric, F.Cu at (143.1, 53.6)
- added R8: 10k, Resistor_SMD:R_0402_1005Metric, F.Cu at (128.1, 54.8)
- added R9: 10k, Resistor_SMD:R_0402_1005Metric, F.Cu at (128.1, 56.8)
- added U10: TPS2051CDBV, Package_TO_SOT_SMD:SOT-23-5, F.Cu at (145.0, 74.4)
- added U11: TPS2051CDBV, Package_TO_SOT_SMD:SOT-23-5, F.Cu at (145.0, 79.0)
- added U12: USB2422/MJ, ROV_PCIe_USB_HUB:QFN-24-1EP_4x4mm_P0.5mm_EP2.5x2.5mm_ThermalVias, F.Cu at (166.9, 61.0)
- added U13: TPS2051CDBV, Package_TO_SOT_SMD:SOT-23-5, F.Cu at (169.9, 50.2)
- added U14: TPS2051CDBV, Package_TO_SOT_SMD:SOT-23-5, F.Cu at (169.9, 54.8)
- added U15: TPS62A02APDDC, Package_TO_SOT_SMD:SOT-23-6, F.Cu at (156.2, 96.2)
- added U16: TPS62A02APDDC, Package_TO_SOT_SMD:SOT-23-6, F.Cu at (156.2, 100.8)
- added U6: USB2422/MJ, ROV_PCIe_USB_HUB:QFN-24-1EP_4x4mm_P0.5mm_EP2.5x2.5mm_ThermalVias, F.Cu at (164.8, 85.2)
- added U7: TPS2051CDBV, Package_TO_SOT_SMD:SOT-23-5, F.Cu at (167.9, 74.4)
- added U8: TPS2051CDBV, Package_TO_SOT_SMD:SOT-23-5, F.Cu at (167.9, 79.0)
- added U9: USB2422/MJ, ROV_PCIe_USB_HUB:QFN-24-1EP_4x4mm_P0.5mm_EP2.5x2.5mm_ThermalVias, F.Cu at (141.9, 85.2)
- added Y1: ABM8-24.000MHZ-B2-T, Crystal:Crystal_SMD_3225-4Pin_3.2x2.5mm, F.Cu at (143.7, 50.1)
- added Y2: ABM8-24.000MHZ-B2-T, Crystal:Crystal_SMD_3225-4Pin_3.2x2.5mm, F.Cu at (129.3, 111.3)
- added Y3: ABM8-24.000MHZ-B2-T, Crystal:Crystal_SMD_3225-4Pin_3.2x2.5mm, F.Cu at (152.2, 89.5)
- added Y4: ABM8-24.000MHZ-B2-T, Crystal:Crystal_SMD_3225-4Pin_3.2x2.5mm, F.Cu at (129.3, 89.5)
- added Y5: ABM8-24.000MHZ-B2-T, Crystal:Crystal_SMD_3225-4Pin_3.2x2.5mm, F.Cu at (154.3, 65.3)
- J1: value USB_A_Stacked -> SFV16R-1STBE1HLF; footprint Connector_USB:USB_A_CUI_UJ2-ADH-TH_Horizontal_Stacked -> ROV_PCIe_USB_HUB:AMPHENOL_SFV16R-1STBE1HLF; moved to B.Cu
- J2, J3, J4: value USB_A_Stacked -> SM04B-SRSS-TB; footprint Connector_USB:USB_A_CUI_UJ2-ADH-TH_Horizontal_Stacked -> Connector_JST:JST_SH_SM04B-SRSS-TB_1x04-1MP_P1.00mm_Horizontal
- U1: value UPD720202K8-7x1-BAA -> MX25V5126FZUI; footprint Package_DFN_QFN:QFN-48-1EP_7x7mm_P0.5mm_EP5.7x5.7mm -> Package_SON:Winbond_USON-8-1EP_3x2mm_P0.5mm_EP0.2x1.6mm
- U2: value USB2514B_Bi -> UPD720201K8-7x1-BAC-A; footprint Package_DFN_QFN:QFN-36-1EP_6x6mm_P0.5mm_EP3.7x3.7mm -> ROV_PCIe_USB_HUB:QFN-68-1EP_8x8mm_P0.4mm_EP6.2x6.2mm
- U3: value USB2514B_Bi -> USB2422/MJ; footprint Package_DFN_QFN:QFN-36-1EP_6x6mm_P0.5mm_EP3.7x3.7mm -> ROV_PCIe_USB_HUB:QFN-24-1EP_4x4mm_P0.5mm_EP2.5x2.5mm_ThermalVias
- U4, U5: value USB2514B_Bi -> TPS2051CDBV; footprint Package_DFN_QFN:QFN-36-1EP_6x6mm_P0.5mm_EP3.7x3.7mm -> Package_TO_SOT_SMD:SOT-23-5
- moved J4 90.1 mm to (154.0, 75.8), turned to 0 degrees
- moved U1 79.0 mm to (142.8, 68.2)
- moved U4 76.5 mm to (145.0, 96.2)
- moved U5 60.4 mm to (145.0, 100.8)
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Connections:
- J1 pad 1: unconnected-(J1-VBUS1-Pad1) -> +5V
- J1 pad 2: unconnected-(J1-D1--Pad2) -> +5V
- J1 pad 3: unconnected-(J1-D1+-Pad3) -> GND
- J1 pad 4: unconnected-(J1-GND1-Pad4) -> PI_PCIE_CLK_P
- J1 pad 5: unconnected-(J1-VBUS2-Pad5) -> PI_PCIE_CLK_N
- J1 pad 6: unconnected-(J1-D2--Pad6) -> GND
- J1 pad 7: unconnected-(J1-D2+-Pad7) -> PI_PCIE_RX_P
- J1 pad 8: unconnected-(J1-GND2-Pad8) -> PI_PCIE_RX_N
- J2 pad 1: unconnected-(J2-VBUS1-Pad1) -> Net-(J2-Pin_1)
- J2 pad 2: unconnected-(J2-D1--Pad2) -> /Hub1/USB1_DN
- J2 pad 3: unconnected-(J2-D1+-Pad3) -> /Hub1/USB1_DP
- J2 pad 4: unconnected-(J2-GND1-Pad4) -> GND
- J3 pad 1: unconnected-(J3-VBUS1-Pad1) -> Net-(J3-Pin_1)
- J3 pad 2: unconnected-(J3-D1--Pad2) -> /Hub1/USB2_DN
- J3 pad 3: unconnected-(J3-D1+-Pad3) -> /Hub1/USB2_DP
- J3 pad 4: unconnected-(J3-GND1-Pad4) -> GND
- J4 pad 1: unconnected-(J4-VBUS1-Pad1) -> Net-(J4-Pin_1)
- J4 pad 2: unconnected-(J4-D1--Pad2) -> /Hub2/USB1_DN
- J4 pad 3: unconnected-(J4-D1+-Pad3) -> /Hub2/USB1_DP
- J4 pad 4: unconnected-(J4-GND1-Pad4) -> GND
- U1 pad 1: unconnected-(U1-PECLKP-Pad1) -> Net-(U1-~{CS})
- U1 pad 2: unconnected-(U1-PECLKN-Pad2) -> Net-(U1-SO)
- U1 pad 3: Net-(U1-AVDD33-Pad25) -> Net-(U1-~{WP})
- U1 pad 4: unconnected-(U1-PETXP-Pad4) -> GND
- U1 pad 5: unconnected-(U1-PETXN-Pad5) -> Net-(U1-SI)
- U1 pad 6: Net-(U1-VDD10-Pad21) -> Net-(U1-SCK)
- U1 pad 8: unconnected-(U1-PERXN-Pad8) -> +3.3V
- U1 pad 9: Net-(U1-VDD10-Pad21) -> GND
- U2 pad 10: unconnected-(U2-VDDA33-Pad10) -> PI_PCIE_TX_P
- U2 pad 11: unconnected-(U2-TEST-Pad11) -> PI_PCIE_TX_N
- U2 pad 12: unconnected-(U2-PRTPWR1/BC_EN1-Pad12) -> +1.05V
- U2 pad 13: unconnected-(U2-OCS_N1-Pad13) -> PCIE_CLKREQ_N
- U2 pad 14: unconnected-(U2-CRFILT-Pad14) -> 1V05_PG
- U2 pad 15: unconnected-(U2-VDD33-Pad15) -> +3.3V
- U2 pad 16: unconnected-(U2-PRTPWR2/BC_EN2-Pad16) -> Net-(U1-SO)
- U2 pad 17: unconnected-(U2-OCS_N2-Pad17) -> Net-(U1-~{CS})
- U2 pad 18: unconnected-(U2-PRTPWR3/BC_EN3-Pad18) -> Net-(U1-SCK)
- U2 pad 19: unconnected-(U2-OCS_N3-Pad19) -> Net-(U1-SI)
- U2 pad 2: unconnected-(U2-USBDP_DN1/PRT_DIS_P1-Pad2) -> PCIE_RST_B
- U2 pad 20: unconnected-(U2-PRTPWR4/BC_EN4-Pad20) -> Net-(U2-OCI1B)
- U2 pad 22: unconnected-(U2-SDA/SMBDATA/NON_REM1-Pad22) -> Net-(U2-OCI1B)
- U2 pad 24: unconnected-(U2-SCL/SMBCLK/CFG_SEL0-Pad24) -> Net-(U2-OCI1B)
- U2 pad 26: unconnected-(U2-RESET_N-Pad26) -> Net-(U2-OCI1B)
- U2 pad 28: unconnected-(U2-SUSP_IND/LOCAL_PWR/NON_REM0-Pad28) -> +1.05V
- U2 pad 29: unconnected-(U2-VDDA33-Pad29) -> +3.3V
- U2 pad 3: unconnected-(U2-USBDM_DN2/PRT_DIS_M2-Pad3) -> PCIE_DET_WAKE
- U2 pad 30: unconnected-(U2-USBDM_UP-Pad30) -> Net-(U2-XT2)
- U2 pad 31: unconnected-(U2-USBDP_UP-Pad31) -> Net-(U2-XT1)
- U2 pad 32: unconnected-(U2-XTALOUT-Pad32) -> /HostController/+3.3V_A
- U2 pad 33: unconnected-(U2-XTALIN/CLKIN-Pad33) -> Net-(U2-RREF)
- U2 pad 34: unconnected-(U2-PLLFILT-Pad34) -> GND
- U2 pad 37: unconnected-(U2-VSS-Pad37) -> +1.05V
- U2 pad 4: unconnected-(U2-USBDP_DN2/PRT_DIS_P2-Pad4) -> PI_PCIE_CLK_P
- U2 pad 5: unconnected-(U2-VDDA33-Pad5) -> PI_PCIE_CLK_N
- U2 pad 6: unconnected-(U2-USBDM_DN3/PRT_DIS_M3-Pad6) -> /HostController/+3.3V_A
- U2 pad 7: unconnected-(U2-USBDP_DN3/PRT_DIS_P3-Pad7) -> /HostController/UPD_PCIE_TX_P
- U2 pad 8: unconnected-(U2-USBDM_DN4/PRT_DIS_M4-Pad8) -> /HostController/UPD_PCIE_TX_N
- U2 pad 9: unconnected-(U2-USBDP_DN4/PRT_DIS_P4-Pad9) -> +1.05V
- U3 pad 1: unconnected-(U3-USBDM_DN1/PRT_DIS_M1-Pad1) -> Net-(C28-Pad1)
- U3 pad 10: unconnected-(U3-VDDA33-Pad10) -> Net-(U3-CRFILT)
- U3 pad 11: unconnected-(U3-TEST-Pad11) -> /Hub1/USB2_PWR_EN
- U3 pad 12: unconnected-(U3-PRTPWR1/BC_EN1-Pad12) -> /Hub1/~{USB2_PWR_OVC}
- U3 pad 13: unconnected-(U3-OCS_N1-Pad13) -> Net-(U3-SMBDATA/NON_REM1)
- U3 pad 14: unconnected-(U3-CRFILT-Pad14) -> GND
- U3 pad 15: unconnected-(U3-VDD33-Pad15) -> 1V05_PG
- U3 pad 16: unconnected-(U3-PRTPWR2/BC_EN2-Pad16) -> VBUS
- U3 pad 17: unconnected-(U3-OCS_N2-Pad17) -> Net-(U3-SUSP_IND/LOCAL_PWR*NON_REM0)
- U3 pad 18: unconnected-(U3-PRTPWR3/BC_EN3-Pad18) -> Net-(C28-Pad1)
- U3 pad 19: unconnected-(U3-OCS_N3-Pad19) -> /USB1_DN
- U3 pad 2: unconnected-(U3-USBDP_DN1/PRT_DIS_P1-Pad2) -> /Hub1/USB1_DN
- U3 pad 20: unconnected-(U3-PRTPWR4/BC_EN4-Pad20) -> /USB1_DP
- U3 pad 21: unconnected-(U3-OCS_N4-Pad21) -> Net-(U3-XTALOUT*(CLKIN_EN))
- U3 pad 22: unconnected-(U3-SDA/SMBDATA/NON_REM1-Pad22) -> Net-(U3-XTALIN/CLKIN)
- U3 pad 23: unconnected-(U3-VDD33-Pad23) -> Net-(U3-PLLFILT)
- U3 pad 24: unconnected-(U3-SCL/SMBCLK/CFG_SEL0-Pad24) -> Net-(U3-RBIAS)
- U3 pad 25: unconnected-(U3-HS_IND/CFG_SEL1-Pad25) -> GND
- U3 pad 3: unconnected-(U3-USBDM_DN2/PRT_DIS_M2-Pad3) -> /Hub1/USB1_DP
- U3 pad 4: unconnected-(U3-USBDP_DN2/PRT_DIS_P2-Pad4) -> /Hub1/USB2_DN
- U3 pad 5: unconnected-(U3-VDDA33-Pad5) -> /Hub1/USB2_DP
- U3 pad 7: unconnected-(U3-USBDP_DN3/PRT_DIS_P3-Pad7) -> /Hub1/USB1_PWR_EN
- U3 pad 8: unconnected-(U3-USBDM_DN4/PRT_DIS_M4-Pad8) -> /Hub1/~{USB1_PWR_OVC}
- U3 pad 9: unconnected-(U3-USBDP_DN4/PRT_DIS_P4-Pad9) -> Net-(C28-Pad1)
- U4 pad 1: unconnected-(U4-USBDM_DN1/PRT_DIS_M1-Pad1) -> Net-(J2-Pin_1)
- U4 pad 2: unconnected-(U4-USBDP_DN1/PRT_DIS_P1-Pad2) -> GND
- U4 pad 3: unconnected-(U4-USBDM_DN2/PRT_DIS_M2-Pad3) -> /Hub1/~{USB1_PWR_OVC}
- U4 pad 4: unconnected-(U4-USBDP_DN2/PRT_DIS_P2-Pad4) -> /Hub1/USB1_PWR_EN
- U4 pad 5: unconnected-(U4-VDDA33-Pad5) -> VBUS
- U5 pad 1: unconnected-(U5-USBDM_DN1/PRT_DIS_M1-Pad1) -> Net-(J3-Pin_1)
- U5 pad 2: unconnected-(U5-USBDP_DN1/PRT_DIS_P1-Pad2) -> GND
- U5 pad 3: unconnected-(U5-USBDM_DN2/PRT_DIS_M2-Pad3) -> /Hub1/~{USB2_PWR_OVC}
- U5 pad 4: unconnected-(U5-USBDP_DN2/PRT_DIS_P2-Pad4) -> /Hub1/USB2_PWR_EN
- U5 pad 5: unconnected-(U5-VDDA33-Pad5) -> VBUS
Routing:
- added copper zone on In1.Cu, net GND
- added copper zone on In2.Cu, net GND
Other:
- outline, holes or cut-outs redrawn
- copper layers 2 -> 4

Commit message: changes
Parts:
- removed FB1, FB2, FB3, FB4, FB5: 220 Ohm @ 100MHz, low DCR, Inductor_SMD:L_0805_2012Metric
- removed J3: SM04B-SRSS-TB, Connector_JST:JST_SH_SM04B-SRSS-TB_1x04-1MP_P1.00mm_Horizontal
- added C67: 10u, Capacitor_SMD:C_0805_2012Metric, F.Cu at (129.2, 106.7)
- added C68: 10u, Capacitor_SMD:C_0805_2012Metric, F.Cu at (129.2, 109.7)
- added C69: 100n, Capacitor_SMD:C_0402_1005Metric, F.Cu at (138.5, 103.6)
- added C70: 100n, Capacitor_SMD:C_0402_1005Metric, F.Cu at (138.5, 105.6)
- added C71: 10p, Capacitor_SMD:C_0402_1005Metric, F.Cu at (138.5, 107.6)
- added C72: 22p, Capacitor_SMD:C_0402_1005Metric, F.Cu at (138.5, 109.5)
- added C73: 22u, Capacitor_SMD:C_1206_3216Metric, F.Cu at (135.0, 97.6)
- added C74: 22u, Capacitor_SMD:C_1206_3216Metric, F.Cu at (135.0, 101.0)
- added D2: SMAJ5.0A, Diode_SMD:D_SMA, F.Cu at (134.7, 91.0)
- added D3: BZX84C10, Package_TO_SOT_SMD:SOT-23, F.Cu at (137.1, 83.3)
- added J10: SM04B-SRSS-TB, Connector_JST:JST_SH_SM04B-SRSS-TB_1x04-1MP_P1.00mm_Horizontal, F.Cu at (149.1, 55.8)
- added J11: SM04B-SRSS-TB, Connector_JST:JST_SH_SM04B-SRSS-TB_1x04-1MP_P1.00mm_Horizontal, F.Cu at (149.1, 63.4)
- added Q1: DMP3018SFV, Package_SON:Diodes_PowerDI3333-8, F.Cu at (137.4, 78.7)
- added R36: 12k, Resistor_SMD:R_0603_1608Metric, F.Cu at (155.6, 55.8)
- added R37: 0, Resistor_SMD:R_0402_1005Metric, F.Cu at (146.2, 68.2)
- added R38: 100k, Resistor_SMD:R_0603_1608Metric, F.Cu at (155.6, 58.3)
- added R39: 100k, Resistor_SMD:R_0603_1608Metric, F.Cu at (155.6, 60.8)
- added R40: 100k, Resistor_SMD:R_0603_1608Metric, F.Cu at (155.6, 63.3)
- added R41: 10k, Resistor_SMD:R_0402_1005Metric, F.Cu at (146.2, 70.2)
- added R42: 10k, Resistor_SMD:R_0402_1005Metric, F.Cu at (146.2, 72.2)
- added R43: 10k, Resistor_SMD:R_0603_1608Metric, F.Cu at (125.0, 97.2)
- added R44: 10k, Resistor_SMD:R_0603_1608Metric, F.Cu at (125.0, 99.7)
- added R45: 453k, Resistor_SMD:R_0603_1608Metric, F.Cu at (125.0, 102.2)
- added R46: 100k, Resistor_SMD:R_0603_1608Metric, F.Cu at (125.0, 104.7)
- added R47: 75k, Resistor_SMD:R_0603_1608Metric, F.Cu at (125.0, 107.2)
- added R48: 100k, Resistor_SMD:R_0603_1608Metric, F.Cu at (125.0, 109.7)
- C1: value 100n -> 330n
- C12, C13, C28, C37, C47, C48: value 100n -> 27p
- C16: value 22u -> 100n; footprint Capacitor_SMD:C_1206_3216Metric -> Capacitor_SMD:C_0402_1005Metric
- C17: value 100n -> 22u; footprint Capacitor_SMD:C_0402_1005Metric -> Capacitor_SMD:C_1206_3216Metric
- C21, C22, C26, C42, C43, C50: value 27p -> 100n
- C23, C33, C49, C59, C60: value 10u -> 100n; footprint Capacitor_SMD:C_0805_2012Metric -> Capacitor_SMD:C_0402_1005Metric
- C30: value 1u -> 100n; footprint Capacitor_SMD:C_0603_1608Metric -> Capacitor_SMD:C_0402_1005Metric
- C31, C61: value 100n -> 1u; footprint Capacitor_SMD:C_0402_1005Metric -> Capacitor_SMD:C_0603_1608Metric
- C34, C35: value 27p -> 10u; footprint Capacitor_SMD:C_0402_1005Metric -> Capacitor_SMD:C_0805_2012Metric
- C36, C44, C45, C55, C56: value 100n -> 10u; footprint Capacitor_SMD:C_0402_1005Metric -> Capacitor_SMD:C_0805_2012Metric
- C38: value 1u -> 27p; footprint Capacitor_SMD:C_0603_1608Metric -> Capacitor_SMD:C_0402_1005Metric
- C41: value 10u -> 1u; footprint Capacitor_SMD:C_0805_2012Metric -> Capacitor_SMD:C_0603_1608Metric
- C46, C54: value 1u -> 10u; footprint Capacitor_SMD:C_0603_1608Metric -> Capacitor_SMD:C_0805_2012Metric
- C51: value 27p -> 1u; footprint Capacitor_SMD:C_0402_1005Metric -> Capacitor_SMD:C_0603_1608Metric
- C57: value 10u -> 27p; footprint Capacitor_SMD:C_0805_2012Metric -> Capacitor_SMD:C_0402_1005Metric
- C58: value 330n -> 27p
- C63: value 10p -> 100n
- C64: value 22p -> 10u; footprint Capacitor_SMD:C_0402_1005Metric -> Capacitor_SMD:C_0805_2012Metric
- C65, C66: value 22u -> 10u; footprint Capacitor_SMD:C_1206_3216Metric -> Capacitor_SMD:C_0805_2012Metric
- J2: value SM04B-SRSS-TB -> 1053131102; footprint Connector_JST:JST_SH_SM04B-SRSS-TB_1x04-1MP_P1.00mm_Horizontal -> ROV_PCIe_USB_HUB:1053131102
- L1, L2: value BDCC00201208R47MWA -> 1u; footprint Inductor_SMD:L_0805_2012Metric -> Inductor_SMD:L_1008_2520Metric
- R1: value 100k -> 10k
- R10: value 1k6 1% -> 10k; footprint Resistor_SMD:R_0603_1608Metric -> Resistor_SMD:R_0402_1005Metric
- R12: value 0 -> 1k6 1%; footprint Resistor_SMD:R_0402_1005Metric -> Resistor_SMD:R_0603_1608Metric
- R13, R28: value 12k -> 10k; footprint Resistor_SMD:R_0603_1608Metric -> Resistor_SMD:R_0402_1005Metric
- R15, R22: value 100k -> 12k
- R16: value 10k -> 0; footprint Resistor_SMD:R_0603_1608Metric -> Resistor_SMD:R_0402_1005Metric
- R18: value 12k -> 100k
- R19, R24: value 0 -> 100k; footprint Resistor_SMD:R_0402_1005Metric -> Resistor_SMD:R_0603_1608Metric
- R2: value 5k1 -> 100k
- R20, R27, R35, R7: value 100k -> 10k; footprint Resistor_SMD:R_0603_1608Metric -> Resistor_SMD:R_0402_1005Metric
- R21: footprint Resistor_SMD:R_0603_1608Metric -> Resistor_SMD:R_0402_1005Metric
- R23: value 12k -> 0; footprint Resistor_SMD:R_0603_1608Metric -> Resistor_SMD:R_0402_1005Metric
- R26: value 453k -> 100k
- R29: value 0 -> 12k; footprint Resistor_SMD:R_0402_1005Metric -> Resistor_SMD:R_0603_1608Metric
- R3: value 10k -> 5k1
- R30: value 100k -> 0; footprint Resistor_SMD:R_0603_1608Metric -> Resistor_SMD:R_0402_1005Metric
- R33: value 10k -> 100k
- R34: value 75k -> 10k; footprint Resistor_SMD:R_0603_1608Metric -> Resistor_SMD:R_0402_1005Metric
- R4: footprint Resistor_SMD:R_0402_1005Metric -> Resistor_SMD:R_0603_1608Metric
- R5, R9: value 10k -> 100k; footprint Resistor_SMD:R_0402_1005Metric -> Resistor_SMD:R_0603_1608Metric
- Y1, Y2, Y3, Y4, Y5: value ABM8-24.000MHZ-B2-T -> ABM11-24.000MHZ-D2X-T; footprint Crystal:Crystal_SMD_3225-4Pin_3.2x2.5mm -> Crystal:Crystal_SMD_2016-4Pin_2.0x1.6mm
- moved R10 83.9 mm to (67.7, 93.0)
- moved R7 83.3 mm to (67.7, 89.0)
- moved C18 80.6 mm to (72.0, 102.8)
- moved C21 79.5 mm to (76.3, 96.8)
- moved C7 79.5 mm to (70.6, 96.8)
- moved C17 78.8 mm to (72.0, 99.5)
- moved C23 75.4 mm to (79.2, 89.0)
- moved C16 72.9 mm to (76.3, 90.9)
- moved R13 72.7 mm to (67.7, 96.9)
- moved U1 72.5 mm to (77.5, 99.7)
- moved C24 71.5 mm to (79.2, 90.9)
- moved C25 71.5 mm to (79.2, 92.9)
- moved C14 70.5 mm to (76.3, 87.0)
- moved C15 70.5 mm to (76.3, 89.0)
- moved C19 70.5 mm to (76.3, 92.9)
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Connections:
- C1 pad 1: +1.05V -> GND
- C1 pad 2: GND -> 1V05_PG
- C10 pad 1: +3.3V -> PI_PCIE_RX_N
- C10 pad 2: GND -> /HostController/UPD_PCIE_TX_N
- C11 pad 1: +3.3V -> +1.05V
- C12 pad 1: +1.05V -> GND
- C12 pad 2: GND -> Net-(C12-Pad2)
- C13 pad 1: +3.3V -> GND
- C13 pad 2: GND -> Net-(U2-XT1)
- C16 pad 1: +3.3V -> +1.05V
- C18 pad 1: +1.05V -> +3.3V
- C19 pad 1: PI_PCIE_RX_P -> +3.3V
- C19 pad 2: /HostController/UPD_PCIE_TX_P -> GND
- C20 pad 1: PI_PCIE_RX_N -> +3.3V
- C20 pad 2: /HostController/UPD_PCIE_TX_N -> GND
- C21 pad 1: GND -> +3.3V
- C21 pad 2: Net-(C21-Pad2) -> GND
- C22 pad 1: GND -> +3.3V
- C22 pad 2: Net-(U2-XT1) -> GND
- C23 pad 1: /HostController/+3.3V_A -> +3.3V
- C24 pad 1: /HostController/+3.3V_A -> +3.3V
- C25 pad 1: /HostController/+3.3V_A -> +3.3V
- C26 pad 1: GND -> +3.3V
- C26 pad 2: Net-(C26-Pad2) -> GND
- C27 pad 2: Net-(U3-XTALOUT*(CLKIN_EN)) -> Net-(C27-Pad2)
- C28 pad 1: Net-(C28-Pad1) -> GND
- C28 pad 2: GND -> Net-(U3-XTALOUT*(CLKIN_EN))
- C29 pad 1: GND -> +3.3V
- C29 pad 2: Net-(U3-PLLFILT) -> GND
- C30 pad 2: Net-(U3-CRFILT) -> Net-(U3-PLLFILT)
- C31 pad 1: Net-(C28-Pad1) -> GND
- C31 pad 2: GND -> Net-(U3-CRFILT)
- C32 pad 1: Net-(C28-Pad1) -> +3.3V
- C33 pad 1: Net-(C28-Pad1) -> +3.3V
- C34 pad 1: GND -> +3.3V
- C34 pad 2: Net-(C34-Pad2) -> GND
- C35 pad 1: GND -> Net-(J4-Pin_1)
- C35 pad 2: Net-(U6-XTALOUT*(CLKIN_EN)) -> GND
- C36 pad 1: Net-(C36-Pad1) -> Net-(J5-Pin_1)
- C37 pad 2: Net-(U6-PLLFILT) -> Net-(C37-Pad2)
- C38 pad 2: Net-(U6-CRFILT) -> Net-(U6-XTALOUT*(CLKIN_EN))
- C39 pad 1: Net-(C36-Pad1) -> +3.3V
- C4 pad 1: +3.3V -> +1.05V
- C40 pad 1: Net-(C36-Pad1) -> GND
- C40 pad 2: GND -> Net-(U6-PLLFILT)
- C41 pad 1: Net-(C36-Pad1) -> GND
- C41 pad 2: GND -> Net-(U6-CRFILT)
- C42 pad 1: GND -> +3.3V
- C42 pad 2: Net-(C42-Pad2) -> GND
- C43 pad 1: GND -> +3.3V
- C43 pad 2: Net-(U9-XTALOUT*(CLKIN_EN)) -> GND
- C44 pad 1: Net-(C44-Pad1) -> +3.3V
- C45 pad 1: GND -> Net-(J6-Pin_1)
- C45 pad 2: Net-(U9-PLLFILT) -> GND
- C46 pad 1: GND -> Net-(J7-Pin_1)
- C46 pad 2: Net-(U9-CRFILT) -> GND
- C47 pad 1: Net-(C44-Pad1) -> GND
- C47 pad 2: GND -> Net-(C47-Pad2)
- C48 pad 1: Net-(C44-Pad1) -> GND
- C48 pad 2: GND -> Net-(U9-XTALOUT*(CLKIN_EN))
- C49 pad 1: Net-(C44-Pad1) -> +3.3V
- C50 pad 2: Net-(C50-Pad2) -> Net-(U9-PLLFILT)
- C51 pad 2: Net-(U12-XTALOUT*(CLKIN_EN)) -> Net-(U9-CRFILT)
- C52 pad 1: Net-(C52-Pad1) -> +3.3V
- C53 pad 1: GND -> +3.3V
- C53 pad 2: Net-(U12-PLLFILT) -> GND
- C54 pad 1: GND -> +3.3V
- C54 pad 2: Net-(U12-CRFILT) -> GND
- C55 pad 1: Net-(C52-Pad1) -> Net-(J8-Pin_1)
- C56 pad 1: Net-(C52-Pad1) -> Net-(J9-Pin_1)
- C57 pad 1: Net-(C52-Pad1) -> GND
- C57 pad 2: GND -> Net-(C57-Pad2)
- C58 pad 2: 1V05_PG -> Net-(U12-XTALOUT*(CLKIN_EN))
- C59 pad 1: +5V -> +3.3V
- C6 pad 1: +3.3V -> +1.05V
- C60 pad 1: +5V -> GND
- C60 pad 2: GND -> Net-(U12-PLLFILT)
- C61 pad 1: +5V -> GND
- C61 pad 2: GND -> Net-(U12-CRFILT)
- C62 pad 1: +5V -> +3.3V
- C63 pad 2: Net-(U15-FB) -> GND
- C64 pad 1: +1.05V -> +3.3V
- C64 pad 2: Net-(U16-FB) -> GND
- C65 pad 1: +3.3V -> Net-(J10-Pin_1)
- C66 pad 1: +1.05V -> Net-(J11-Pin_1)
- C8 pad 1: +3.3V -> +1.05V
- C9 pad 1: +1.05V -> PI_PCIE_RX_P
- C9 pad 2: GND -> /HostController/UPD_PCIE_TX_P
- J2 pad 1: Net-(J2-Pin_1) -> GND
- J2 pad 2: /Hub1/USB1_DN -> Net-(D2-A1)
- J4 pad 2: /Hub2/USB1_DN -> /Hub1/USB1_DN
- J4 pad 3: /Hub2/USB1_DP -> /Hub1/USB1_DP
- J5 pad 2: /Hub2/USB2_DN -> /Hub1/USB2_DN
- J5 pad 3: /Hub2/USB2_DP -> /Hub1/USB2_DP
- J6 pad 2: /Hub3/USB1_DN -> /Hub2/USB1_DN
- J6 pad 3: /Hub3/USB1_DP -> /Hub2/USB1_DP
- J7 pad 2: /Hub3/USB2_DN -> /Hub2/USB2_DN
- J7 pad 3: /Hub3/USB2_DP -> /Hub2/USB2_DP
- J8 pad 2: /Hub4/USB1_DN -> /Hub3/USB1_DN
- J8 pad 3: /Hub4/USB1_DP -> /Hub3/USB1_DP
- J9 pad 2: /Hub4/USB2_DN -> /Hub3/USB2_DN
- J9 pad 3: /Hub4/USB2_DP -> /Hub3/USB2_DP
- R1 pad 1: PCIE_PWR_EN -> +3.3V
- R1 pad 2: GND -> 1V05_PG
- R10 pad 1: GND -> +3.3V
- R10 pad 2: Net-(U2-RREF) -> Net-(U1-SI)
- R11 pad 2: Net-(U2-OCI1B) -> Net-(U1-~{CS})
- R12 pad 1: Net-(C21-Pad2) -> GND
- R12 pad 2: Net-(U2-XT2) -> Net-(U2-RREF)
- R13 pad 1: GND -> +3.3V
- R13 pad 2: Net-(U3-RBIAS) -> Net-(U2-OCI1B)
- R14 pad 1: Net-(C26-Pad2) -> Net-(C12-Pad2)
- R14 pad 2: Net-(U3-XTALIN/CLKIN) -> Net-(U2-XT2)
- R15 pad 1: Net-(U3-SUSP_IND/LOCAL_PWR*NON_REM0) -> GND
- R15 pad 2: GND -> Net-(U3-RBIAS)
- R16 pad 1: +3.3V -> Net-(C27-Pad2)
- R16 pad 2: 3V3_PG -> Net-(U3-XTALIN/CLKIN)
- R17 pad 1: Net-(U3-SMBDATA/NON_REM1) -> Net-(U3-SUSP_IND/LOCAL_PWR*NON_REM0)
- R18 pad 1: GND -> Net-(U3-SMBCLK/CFG_SEL0)
- R18 pad 2: Net-(U6-RBIAS) -> GND
- R19 pad 1: Net-(C34-Pad2) -> Net-(U3-SMBDATA/NON_REM1)
- R19 pad 2: Net-(U6-XTALIN/CLKIN) -> GND
- R2 pad 1: +5V -> PCIE_PWR_EN
- R2 pad 2: PCIE_DET_WAKE -> GND
- R20 pad 1: Net-(U6-SUSP_IND/LOCAL_PWR*NON_REM0) -> +3.3V
- R20 pad 2: GND -> /Hub1/~{USB1_PWR_OVC}
- R21 pad 2: 1V05_PG -> /Hub1/~{USB2_PWR_OVC}
- R22 pad 1: Net-(U6-SMBDATA/NON_REM1) -> GND
- R22 pad 2: GND -> Net-(U6-RBIAS)
- R23 pad 1: GND -> Net-(C37-Pad2)
- R23 pad 2: Net-(U9-RBIAS) -> Net-(U6-XTALIN/CLKIN)
- R24 pad 1: Net-(C42-Pad2) -> Net-(U6-SUSP_IND/LOCAL_PWR*NON_REM0)
- R24 pad 2: Net-(U9-XTALIN/CLKIN) -> GND
- R25 pad 1: Net-(U9-SUSP_IND/LOCAL_PWR*NON_REM0) -> Net-(U6-SMBCLK/CFG_SEL0)
- R26 pad 1: +3.3V -> Net-(U6-SMBDATA/NON_REM1)
- R26 pad 2: Net-(U15-FB) -> GND
- R27 pad 1: Net-(U9-SMBDATA/NON_REM1) -> +3.3V
- R27 pad 2: GND -> /Hub2/~{USB1_PWR_OVC}
- R28 pad 1: GND -> +3.3V
- R28 pad 2: Net-(U12-RBIAS) -> /Hub2/~{USB2_PWR_OVC}
- R29 pad 1: Net-(C50-Pad2) -> GND
- R29 pad 2: Net-(U12-XTALIN/CLKIN) -> Net-(U9-RBIAS)
- R3 pad 1: PCIE_DET_WAKE -> +5V
- R3 pad 2: GND -> PCIE_DET_WAKE
- R30 pad 1: Net-(U12-SUSP_IND/LOCAL_PWR*NON_REM0) -> Net-(C47-Pad2)
- R30 pad 2: GND -> Net-(U9-XTALIN/CLKIN)
- R31 pad 1: Net-(U15-FB) -> Net-(U9-SUSP_IND/LOCAL_PWR*NON_REM0)
- R32 pad 1: Net-(U12-SMBDATA/NON_REM1) -> Net-(U9-SMBCLK/CFG_SEL0)
- R33 pad 1: +3.3V -> Net-(U9-SMBDATA/NON_REM1)
- R33 pad 2: 1V05_PG -> GND
- R34 pad 1: +1.05V -> +3.3V
- R34 pad 2: Net-(U16-FB) -> /Hub3/~{USB1_PWR_OVC}
- R35 pad 1: Net-(U16-FB) -> +3.3V
- R35 pad 2: GND -> /Hub3/~{USB2_PWR_OVC}
- R4 pad 1: +3.3V -> PCIE_DET_WAKE
- R4 pad 2: PCIE_CLKREQ_N -> GND
- R5 pad 1: +3.3V -> Net-(D3A-A)
- R5 pad 2: Net-(U1-~{WP}) -> GND
- R6 pad 2: Net-(U1-SO) -> PCIE_CLKREQ_N
- R7 pad 1: Net-(U1-SCK) -> +3.3V
- R7 pad 2: GND -> Net-(U1-~{WP})
- R8 pad 2: Net-(U1-SI) -> Net-(U1-SO)
- R9 pad 1: +3.3V -> Net-(U1-SCK)
- R9 pad 2: Net-(U1-~{CS}) -> GND
- U10 pad 1: Net-(J6-Pin_1) -> Net-(J8-Pin_1)
- U11 pad 1: Net-(J7-Pin_1) -> Net-(J9-Pin_1)
- U12 pad 1: Net-(C52-Pad1) -> +3.3V
- U12 pad 14: GND -> Net-(U12-SMBCLK/CFG_SEL0)
- U12 pad 16: VBUS -> +3.3V
- U12 pad 18: Net-(C52-Pad1) -> +3.3V
- U12 pad 9: Net-(C52-Pad1) -> +3.3V
- U13 pad 1: Net-(J8-Pin_1) -> Net-(J10-Pin_1)
- U14 pad 1: Net-(J9-Pin_1) -> Net-(J11-Pin_1)
- U2 pad 32: /HostController/+3.3V_A -> +3.3V
- U2 pad 6: /HostController/+3.3V_A -> +3.3V
- U3 pad 1: Net-(C28-Pad1) -> +3.3V
- U3 pad 14: GND -> Net-(U3-SMBCLK/CFG_SEL0)
- U3 pad 16: VBUS -> +3.3V
- U3 pad 18: Net-(C28-Pad1) -> +3.3V
- U3 pad 9: Net-(C28-Pad1) -> +3.3V
- U4 pad 1: Net-(J2-Pin_1) -> Net-(J4-Pin_1)
- U5 pad 1: Net-(J3-Pin_1) -> Net-(J5-Pin_1)
- U6 pad 1: Net-(C36-Pad1) -> +3.3V
- U6 pad 14: GND -> Net-(U6-SMBCLK/CFG_SEL0)
- U6 pad 16: VBUS -> +3.3V
- U6 pad 18: Net-(C36-Pad1) -> +3.3V
- U6 pad 9: Net-(C36-Pad1) -> +3.3V
- U7 pad 1: Net-(J4-Pin_1) -> Net-(J6-Pin_1)
- U8 pad 1: Net-(J5-Pin_1) -> Net-(J7-Pin_1)
- U9 pad 1: Net-(C44-Pad1) -> +3.3V
- U9 pad 14: GND -> Net-(U9-SMBCLK/CFG_SEL0)
- U9 pad 16: VBUS -> +3.3V
- U9 pad 18: Net-(C44-Pad1) -> +3.3V
- U9 pad 9: Net-(C44-Pad1) -> +3.3V
- Y1 pad 1: Net-(C21-Pad2) -> Net-(C12-Pad2)
- Y2 pad 1: Net-(C26-Pad2) -> Net-(C27-Pad2)
- Y3 pad 1: Net-(C34-Pad2) -> Net-(C37-Pad2)
- Y4 pad 1: Net-(C42-Pad2) -> Net-(C47-Pad2)
- Y5 pad 1: Net-(C50-Pad2) -> Net-(C57-Pad2)
Routing:
- net GND: track 0.00 -> 2.76 mm
- net Net-(C12-Pad2): track 0.00 -> 1.40 mm
- net Net-(U2-XT1): track 0.00 -> 1.36 mm

Commit message: work
Parts:
- removed the C16 at (76.3, 90.9)
- removed the C36 at (155.8, 95.7)
- removed the C4 at (70.6, 90.9)
- removed the C66 at (155.8, 72.1)
- removed the R21 at (146.2, 95.8)
- removed the R23 at (169.0, 91.8)
- removed the R39 at (155.6, 60.8)
- removed the R40 at (155.6, 63.3)
- removed the R41 at (146.2, 70.2)
- removed the R42 at (146.2, 72.2)
- added C15: 100n, Capacitor_SMD:C_0402_1005Metric, F.Cu at (65.7, 77.6)
- added C26: 10p, Capacitor_SMD:C_0402_1005Metric, F.Cu at (126.4, 100.6)
- added C46: 10p, Capacitor_SMD:C_0402_1005Metric, F.Cu at (84.1, 32.1)
- added R27: 12k, Resistor_SMD:R_0603_1608Metric, F.Cu at (86.9, 35.5)
- added R28: 100k, Resistor_SMD:R_0603_1608Metric, F.Cu at (89.4, 35.5)
- C11: renamed from C12; value 27p -> 10p
- C12: renamed from C13; value 27p -> 10p
- C27, C47, C57: value 27p -> 10p
- C28, C48, C58: value 27p -> 100n
- C30, C50, C60: value 100n -> 1u; footprint Capacitor_SMD:C_0402_1005Metric -> Capacitor_SMD:C_0603_1608Metric
- C31, C51, C61: value 1u -> 100n; footprint Capacitor_SMD:C_0603_1608Metric -> Capacitor_SMD:C_0402_1005Metric
- C33, C53, C63: value 100n -> 10u; footprint Capacitor_SMD:C_0402_1005Metric -> Capacitor_SMD:C_0805_2012Metric
- C36: renamed from C37; value 27p -> 10p
- C37: renamed from C38; value 27p -> 10p
- C56: value 10u -> 10p; footprint Capacitor_SMD:C_0805_2012Metric -> Capacitor_SMD:C_0402_1005Metric
- R16, R30: value 0 -> 100k; footprint Resistor_SMD:R_0402_1005Metric -> Resistor_SMD:R_0603_1608Metric
- R19, R31, R32, R38: value 100k -> 10k; footprint Resistor_SMD:R_0603_1608Metric -> Resistor_SMD:R_0402_1005Metric
- R29, R36: value 12k -> 100k
- R33: value 100k -> 12k
- R34, R35: value 10k -> 100k; footprint Resistor_SMD:R_0402_1005Metric -> Resistor_SMD:R_0603_1608Metric
- R37: value 0 -> 10k
- Y1, Y2, Y3, Y4, Y5: value ABM11-24.000MHZ-D2X-T -> ECS-240-8-37B-CKY-TR
- moved C56 128.1 mm to (57.0, 31.7), turned to 90 degrees
- moved R33 121.9 mm to (59.8, 35.1), turned to 90 degrees
- moved R34 112.3 mm to (62.3, 35.1), turned to 90 degrees
- moved R35 110.6 mm to (64.8, 35.1), turned to 90 degrees
- moved C60 104.4 mm to (57.3, 35.1), turned to 90 degrees
- moved C57 102.2 mm to (59.0, 31.7), turned to 90 degrees
- moved C58 100.7 mm to (61.0, 31.7), turned to 90 degrees
- moved U11 100.7 mm to (85.2, 58.0)
- moved C50 100.3 mm to (84.4, 35.5), turned to 90 degrees
- moved U12 99.4 mm to (62.3, 63.6), turned to -90 degrees
- moved C59 99.3 mm to (63.0, 31.7), turned to 90 degrees
- moved U9 99.2 mm to (85.3, 64.0), turned to -90 degrees
- moved C47 98.1 mm to (86.1, 32.1), turned to 90 degrees
- moved U14 97.7 mm to (65.3, 58.0)
- moved C55 97.3 mm to (82.0, 58.2), turned to -90 degrees
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- renumbered C11 to C10, C14 to C13, C15 to C14, C17 to C16, C18 to C17, C19 to C18, C20 to C19, C21 to C20, C22 to C21, C23 to C22, C24 to C23, C25 to C24, C26 to C25, C39 to C38, C40 to C39, C5 to C4, C41 to C40, C42 to C41, C43 to C42, C44 to C43, C45 to C44, C46 to C45, C6 to C5, C7 to C6, C67 to C66, C68 to C67, C69 to C68, C70 to C69, C8 to C7, C71 to C70, C72 to C71, C73 to C72, C74 to C73, C9 to C8, C10 to C9, R22 to R21, R24 to R22, R25 to R23, R26 to R24, R27 to R25, R28 to R26, R43 to R39, R44 to R40, R45 to R41, R46 to R42, R47 to R43, R48 to R44
Connections:
- C27 pad 2: Net-(C27-Pad2) -> Net-(U3-XTALOUT*(CLKIN_EN))
- C28 pad 1: GND -> +3.3V
- C28 pad 2: Net-(U3-XTALOUT*(CLKIN_EN)) -> GND
- C29 pad 1: +3.3V -> GND
- C29 pad 2: GND -> Net-(U3-PLLFILT)
- C30 pad 2: Net-(U3-PLLFILT) -> Net-(U3-CRFILT)
- C31 pad 1: GND -> +3.3V
- C31 pad 2: Net-(U3-CRFILT) -> GND
- C34 pad 1: +3.3V -> Net-(J4-Pin_1)
- C35 pad 1: Net-(J4-Pin_1) -> Net-(J5-Pin_1)
- C36 pad 2: Net-(C37-Pad2) -> Net-(U6-XTALIN/CLKIN)
- C47 pad 2: Net-(C47-Pad2) -> Net-(U9-XTALOUT*(CLKIN_EN))
- C48 pad 1: GND -> +3.3V
- C48 pad 2: Net-(U9-XTALOUT*(CLKIN_EN)) -> GND
- C49 pad 1: +3.3V -> GND
- C49 pad 2: GND -> Net-(U9-PLLFILT)
- C50 pad 2: Net-(U9-PLLFILT) -> Net-(U9-CRFILT)
- C51 pad 1: GND -> +3.3V
- C51 pad 2: Net-(U9-CRFILT) -> GND
- C54 pad 1: +3.3V -> Net-(J8-Pin_1)
- C55 pad 1: Net-(J8-Pin_1) -> Net-(J9-Pin_1)
- C56 pad 1: Net-(J9-Pin_1) -> GND
- C56 pad 2: GND -> Net-(U12-XTALIN/CLKIN)
- C57 pad 2: Net-(C57-Pad2) -> Net-(U12-XTALOUT*(CLKIN_EN))
- C58 pad 1: GND -> +3.3V
- C58 pad 2: Net-(U12-XTALOUT*(CLKIN_EN)) -> GND
- C59 pad 1: +3.3V -> GND
- C59 pad 2: GND -> Net-(U12-PLLFILT)
- C60 pad 2: Net-(U12-PLLFILT) -> Net-(U12-CRFILT)
- C61 pad 1: GND -> +3.3V
- C61 pad 2: Net-(U12-CRFILT) -> GND
- C64 pad 1: +3.3V -> Net-(J10-Pin_1)
- C65 pad 1: Net-(J10-Pin_1) -> Net-(J11-Pin_1)
- C8 pad 1: PI_PCIE_RX_P -> PI_PCIE_RX_N
- C9 pad 1: PI_PCIE_RX_N -> PI_PCIE_RX_P
- R16 pad 1: Net-(C27-Pad2) -> Net-(U3-SUSP_IND/LOCAL_PWR*NON_REM0)
- R16 pad 2: Net-(U3-XTALIN/CLKIN) -> GND
- R17 pad 1: Net-(U3-SUSP_IND/LOCAL_PWR*NON_REM0) -> Net-(U3-SMBCLK/CFG_SEL0)
- R18 pad 1: Net-(U3-SMBCLK/CFG_SEL0) -> Net-(U3-SMBDATA/NON_REM1)
- R19 pad 1: Net-(U3-SMBDATA/NON_REM1) -> +3.3V
- R19 pad 2: GND -> /Hub1/~{USB1_PWR_OVC}
- R20 pad 2: /Hub1/~{USB1_PWR_OVC} -> /Hub1/~{USB2_PWR_OVC}
- R29 pad 1: GND -> Net-(U9-SMBCLK/CFG_SEL0)
- R29 pad 2: Net-(U9-RBIAS) -> GND
- R30 pad 1: Net-(C47-Pad2) -> Net-(U9-SMBDATA/NON_REM1)
- R30 pad 2: Net-(U9-XTALIN/CLKIN) -> GND
- R31 pad 1: Net-(U9-SUSP_IND/LOCAL_PWR*NON_REM0) -> +3.3V
- R31 pad 2: GND -> /Hub3/~{USB1_PWR_OVC}
- R32 pad 1: Net-(U9-SMBCLK/CFG_SEL0) -> +3.3V
- R32 pad 2: GND -> /Hub3/~{USB2_PWR_OVC}
- R33 pad 1: Net-(U9-SMBDATA/NON_REM1) -> GND
- R33 pad 2: GND -> Net-(U12-RBIAS)
- R34 pad 1: +3.3V -> Net-(U12-SUSP_IND/LOCAL_PWR*NON_REM0)
- R34 pad 2: /Hub3/~{USB1_PWR_OVC} -> GND
- R35 pad 1: +3.3V -> Net-(U12-SMBCLK/CFG_SEL0)
- R35 pad 2: /Hub3/~{USB2_PWR_OVC} -> GND
- R36 pad 1: GND -> Net-(U12-SMBDATA/NON_REM1)
- R36 pad 2: Net-(U12-RBIAS) -> GND
- R37 pad 1: Net-(C57-Pad2) -> +3.3V
- R37 pad 2: Net-(U12-XTALIN/CLKIN) -> /Hub4/~{USB1_PWR_OVC}
- R38 pad 1: Net-(U12-SUSP_IND/LOCAL_PWR*NON_REM0) -> +3.3V
- R38 pad 2: GND -> /Hub4/~{USB2_PWR_OVC}
- U2 pad 4: PI_PCIE_CLK_P -> PI_PCIE_CLK_N
- U2 pad 5: PI_PCIE_CLK_N -> PI_PCIE_CLK_P
- U2 pad 64: unconnected-(U2-U3RXDP4-Pad64) -> GND
- U2 pad 65: unconnected-(U2-U3RXDN4-Pad65) -> GND
- Y2 pad 1: Net-(C27-Pad2) -> Net-(U3-XTALIN/CLKIN)
- Y3 pad 1: Net-(C37-Pad2) -> Net-(U6-XTALIN/CLKIN)
- Y4 pad 1: Net-(C47-Pad2) -> Net-(U9-XTALIN/CLKIN)
- Y5 pad 1: Net-(C57-Pad2) -> Net-(U12-XTALIN/CLKIN)
Routing:
- net +3.3V: track 0.00 -> 152.2 mm, vias 0 -> 28
- net GND: track 2.76 -> 147.2 mm, vias 0 -> 80
- net VBUS: track 0.00 -> 101.7 mm, vias 0 -> 8
- net +5V: track 0.00 -> 96.6 mm, vias 0 -> 10
- net 1V05_PG: track 0.00 -> 56.6 mm, vias 0 -> 3
- net +1.05V: track 0.00 -> 45.7 mm, vias 0 -> 17
- net PCIE_PWR_EN: track 0.00 -> 42.3 mm, vias 0 -> 2
- net Net-(U1-SCK): track 0.00 -> 25.2 mm, vias 0 -> 2
- net PCIE_CLKREQ_N: track 0.00 -> 23.3 mm, vias 0 -> 1
- net Net-(U1-SI): track 0.00 -> 21.0 mm, vias 0 -> 2
- net PI_PCIE_TX_N: track 0.00 -> 18.9 mm, vias 0 -> 1
- net PI_PCIE_TX_P: track 0.00 -> 17.7 mm, vias 0 -> 1
- net Net-(U1-SO): track 0.00 -> 16.8 mm, vias 0 -> 2
- net Net-(U1-~{CS}): track 0.00 -> 16.5 mm, vias 0 -> 2
- net 3V3_PG: track 0.00 -> 14.6 mm, vias 0 -> 2
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- added copper zone on B.Cu, net +1.05V
- added copper zone on F.Cu, net +1.05V
- added copper zone on In2.Cu, net +1.05V
- added copper zone on B.Cu, net +3.3V
- added copper zone on F.Cu, net +3.3V
- added copper zone on In2.Cu, net +3.3V
- added copper zone on B.Cu, net +5V
- added copper zone on F.Cu, net +5V
- added copper zone on F.Cu, net GND
- added copper zone on F.Cu, net Net-(D2-A1)
- added copper zone on F.Cu, net Net-(U15-SW)
- added copper zone on F.Cu, net Net-(U16-SW)
- added copper zone on F.Cu, net VBUS

Commit message: changes
Parts:
- moved U3 56.7 mm to (130.5, 130.1), turned to 0 degrees
- moved C35 53.1 mm to (124.8, 134.5), turned to 0 degrees
- moved Y2 52.2 mm to (115.7, 131.4), turned to 0 degrees
- moved R20 51.7 mm to (119.2, 132.6), turned to 0 degrees
- moved R19 48.0 mm to (119.2, 130.6), turned to 0 degrees
- moved U5 47.7 mm to (132.0, 121.4), turned to 0 degrees
- moved J5 47.5 mm to (118.1, 125.8), turned to 0 degrees
- moved C34 47.2 mm to (124.8, 131.5), turned to 0 degrees
- moved C33 41.2 mm to (124.8, 128.4), turned to 0 degrees
- moved U4 36.6 mm to (132.0, 116.8), turned to 0 degrees
- moved R18 35.8 mm to (124.5, 125.7), turned to 0 degrees
- moved U11 35.1 mm to (108.6, 31.8)
- moved C32 34.5 mm to (128.0, 125.2), turned to 0 degrees
- moved U10 34.2 mm to (108.6, 27.2)
- moved U9 32.1 mm to (107.1, 40.5), turned to 0 degrees
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Routing:
- net +3.3V: track 152.2 -> 162.5 mm, vias 28 -> 29
- net +1.05V: track 45.7 -> 49.7 mm, vias 17 -> 18
- net Net-(U1-SI): track 21.0 -> 19.1 mm, vias 2 -> 0
- net Net-(U1-SCK): track 25.2 -> 23.3 mm, vias 2 -> 0
- net Net-(U1-~{CS}): track 16.5 -> 14.7 mm, vias 2 -> 0
- net Net-(U1-SO): track 16.8 -> 15.4 mm, vias 2 -> 0
- net GND: track 147.2 -> 146.4 mm, vias 80 -> 79
- net 1V05_PG: track 56.6 -> 55.9 mm
