File: ROV_PCIe_USB_HUB_FINAL/ROV_PCIE_USB_HUB_FINAL.kicad_pcb (KiCad board)
At the start: 4 copper layers, 65 x 56.5 mm, 158 parts, among them J1 SFV16R-1STBE1HLF, J10 SM04B-SRSS-TB, J11 SM04B-SRSS-TB, J2 1053131102, J4 SM04B-SRSS-TB, J5 SM04B-SRSS-TB, J6 SM04B-SRSS-TB, J7 SM04B-SRSS-TB, J8 SM04B-SRSS-TB, J9 SM04B-SRSS-TB, Q1 DMP3018SFV, U1 MX25V5126FZUI, U10 TPS2051CDBV, U11 TPS2051CDBV, U12 USB2422/MJ, U13 TPS2051CDBV, U14 TPS2051CDBV, U15 TPS62A02APDDC, U16 TPS62A02APDDC, U2 UPD720201K8-7x1-BAC-A, U3 USB2422/MJ, U4 TPS2051CDBV, U5 TPS2051CDBV, U6 USB2422/MJ, U7 TPS2051CDBV, U8 TPS2051CDBV, U9 USB2422/MJ, Y1 ECS-240-8-37B-CKY-TR, Y2 ECS-240-8-37B-CKY-TR, Y3 ECS-240-8-37B-CKY-TR, Y4 ECS-240-8-37B-CKY-TR, Y5 ECS-240-8-37B-CKY-TR

Commit message: reroute
Parts:
- added J12: Raspberry_Pi_4, Connector_PinSocket_2.54mm:PinSocket_2x20_P2.54mm_Vertical, B.Cu at (58.5, 54.8)
- moved U3 74.7 mm to (65.3, 93.8), turned to 90 degrees
- moved R1 67.3 mm to (17.5, 73.5), turned to 0 degrees
- moved C26 66.5 mm to (61.6, 111.2)
- moved C27 66.5 mm to (61.6, 113.1)
- moved C28 66.5 mm to (61.6, 115.1)
- moved C29 66.5 mm to (61.6, 117.1)
- moved C30 66.5 mm to (58.1, 111.4)
- moved C31 66.5 mm to (61.6, 119.0)
- moved C32 66.5 mm to (61.6, 121.0)
- moved C33 66.5 mm to (58.4, 124.2)
- moved C34 66.5 mm to (58.4, 127.2)
- moved C35 66.5 mm to (58.4, 130.3)
- moved R15 66.5 mm to (58.1, 114.0)
- moved R16 66.5 mm to (58.1, 116.5)
- moved R17 66.5 mm to (58.1, 119.0)
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Connections:
- C8 pad 1: PI_PCIE_RX_N -> PI_PCIE_RX_P
- C9 pad 1: PI_PCIE_RX_P -> PI_PCIE_RX_N
- U2 pad 4: PI_PCIE_CLK_N -> PI_PCIE_CLK_P
- U2 pad 5: PI_PCIE_CLK_P -> PI_PCIE_CLK_N
Routing:
- net +3.3V: track 162.5 -> 36.3 mm, vias 29 -> 23
- net VBUS: track 101.7 -> 7.31 mm
- net +5V: track 96.6 -> 7.23 mm, vias 10 -> 8
- net PI_PCIE_CLK_P: track 12.4 -> 64.0 mm
- net PI_PCIE_CLK_N: track 12.4 -> 62.3 mm
- net PI_PCIE_RX_P: track 3.47 -> 48.7 mm
- net PI_PCIE_RX_N: track 3.47 -> 47.0 mm
- net PCIE_PWR_EN: track 42.3 -> 1.30 mm, vias 2 -> 1
- net 1V05_PG: track 55.9 -> 17.7 mm, vias 3 -> 1
- net +1.05V: track 49.7 -> 17.6 mm, vias 18 -> 16
- net /USB1_DP: track 5.84 -> 36.8 mm
- net /USB1_DN: track 6.26 -> 36.3 mm
- net PI_PCIE_TX_P: track 17.7 -> 45.0 mm
- net Net-(J12-3V3-Pad1): track 0.00 -> 25.1 mm
- net PI_PCIE_TX_N: track 18.9 -> 43.4 mm
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
Commit message: changes
Parts:
- moved C1 46.2 mm to (64.9, 82.3)
- moved D1 46.2 mm to (62.8, 80.7)
- moved R1 46.2 mm to (62.8, 82.7)
- moved R20 39.9 mm to (68.0, 91.5), turned to 180 degrees
- moved C51 37.4 mm to (97.5, 86.1), turned to 180 degrees
- moved C47 36.8 mm to (98.6, 88.8), turned to -90 degrees
- moved C53 36.6 mm to (97.5, 80.0), turned to 180 degrees
- moved C33 36.3 mm to (67.6, 89.2), turned to 90 degrees
- moved Y2 36.1 mm to (58.4, 92.3), turned to 90 degrees
- moved R30 35.5 mm to (97.0, 81.8), turned to 180 degrees
- moved R19 35.0 mm to (68.0, 94.9), turned to 180 degrees
- moved R29 34.8 mm to (97.0, 83.3), turned to 180 degrees
- moved R28 34.5 mm to (97.0, 84.9), turned to 180 degrees
- moved C52 34.2 mm to (102.3, 79.6), turned to 90 degrees
- moved R18 33.8 mm to (65.8, 88.6), turned to 90 degrees
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Routing:
- net 1V05_PG: track 17.7 -> 124.7 mm, vias 1 -> 9
- net +3.3V: track 36.3 -> 113.1 mm, vias 23 -> 55
- net GND: track 124.6 -> 191.7 mm, vias 66 -> 202
- net PCIE_DET_WAKE: track 3.57 -> 43.9 mm, vias 1 -> 3
- net PCIE_RST_B: track 3.67 -> 43.3 mm
- net PCIE_CLKREQ_N: track 4.49 -> 41.3 mm, vias 0 -> 3
- net PCIE_PWR_EN: track 1.30 -> 22.3 mm, vias 1 -> 3
- net /Hub1/~{USB1_PWR_OVC}: track 0.00 -> 13.7 mm, vias 0 -> 2
- net /Hub3/~{USB1_PWR_OVC}: track 0.00 -> 13.7 mm, vias 0 -> 2
- net /USB3_DP: track 12.7 -> 25.7 mm
- net /Hub1/USB1_PWR_EN: track 0.00 -> 12.7 mm, vias 0 -> 2
- net /Hub3/USB1_PWR_EN: track 0.00 -> 12.7 mm, vias 0 -> 2
- net +5V: track 7.23 -> 19.8 mm, vias 8 -> 10
- net /USB3_DN: track 12.7 -> 25.1 mm
- net /Hub4/USB1_PWR_EN: track 1.19 -> 12.7 mm, vias 1 -> 2
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- added copper zone on In2.Cu, net +5V
- added copper zone on In2.Cu, net VBUS
- removed copper zone on B.Cu, net +1.05V
- removed copper zone on B.Cu, net +3.3V
- removed copper zone on F.Cu, net +5V

Commit message: add images, clean up
Parts:
- added G*** (x2): LOGO, LOGO, F.Cu at (91.5, 65.0)
- added G***: LOGO, LOGO, B.Cu at (90.5, 84.0)
Other:
- board text added: "Purdue ROV RPi 5 PCIe USB Root Hub Sam Nadol https://snadol.com"
