File: ROV_PCIe_USB_HUB_FINAL/ROV_PCIE_USB_HUB_FINAL.kicad_sch (KiCad schematic)
At the start: 13 parts, among them J1 USB_A_Stacked, J2 USB_A_Stacked, J3 USB_A_Stacked, J4 USB_A_Stacked, U1 UPD720202K8-7x1-BAA, U2 USB2514B_Bi, U3 USB2514B_Bi, U4 USB2514B_Bi, U5 USB2514B_Bi

Commit message: work
Parts:
- removed J1, J2, J3, J4: USB_A_Stacked, Connector_USB:USB_A_CUI_UJ2-ADH-TH_Horizontal_Stacked, symbol Connector:USB_A_Stacked
- removed U1: UPD720202K8-7x1-BAA, Package_DFN_QFN:QFN-48-1EP_7x7mm_P0.5mm_EP5.7x5.7mm, symbol Interface_USB:UPD720202K8-7x1-BAA
- removed U2, U3, U4, U5: USB2514B_Bi, Package_DFN_QFN:QFN-36-1EP_6x6mm_P0.5mm_EP3.7x3.7mm, symbol Interface_USB:USB2514B_Bi
- added C58: 330n, Capacitor_SMD:C_0402_1005Metric, symbol Device:C_Small
- added D1: BAT54W, Package_TO_SOT_SMD:SOT-323_SC-70, symbol Diode:BAT54W
- added J1: SFV16R-1STBE1HLF, ROV_PCIe_USB_HUB:AMPHENOL_SFV16R-1STBE1HLF, symbol ROV_PCIe_USB_HUB:SFV16R-1STBE1HLF
- added R1: 100k, Resistor_SMD:R_0603_1608Metric, symbol Device:R_Small_US
- added R2: 5k1, Resistor_SMD:R_0603_1608Metric, symbol Device:R_Small_US
- added R3, R33: 10k, Resistor_SMD:R_0603_1608Metric, symbol Device:R_Small_US
Connections:
- new net: J1.SH1 (SH), J1.SH2 (SH)
- new net +3.3V: D1.3 (K), R33.1
- new net +5V: J1.1, J1.2, R2.1
- new net 1V05_PG: C58.2, D1.1 (A), R33.2
- new net GND: C58.1, J1.12, J1.3, J1.6, J1.9, R1.2, R3.2
- new net PCIE_CLKREQ_N: J1.15
- new net PCIE_DET_WAKE: J1.14, R2.2, R3.1
- new net PCIE_PWR_EN: J1.13, R1.1
- new net PCIE_RST_B: J1.16
- new net PI_PCIE_CLK_N: J1.5
- new net PI_PCIE_CLK_P: J1.4
- new net PI_PCIE_RX_N: J1.8
- new net PI_PCIE_RX_P: J1.7
- new net PI_PCIE_TX_N: J1.11
- new net PI_PCIE_TX_P: J1.10
- no-connect marks 4 -> 5
Other:
- added sheet HostController (HostController.kicad_sch)
- added sheet Hub1 (Hub1.kicad_sch)
- added sheet Hub2 (Hub1.kicad_sch)
- added sheet Hub3 (Hub1.kicad_sch)
- added sheet Hub4 (Hub1.kicad_sch)
- added sheet Power (Power.kicad_sch)

Commit message: changes
Parts:
- added D2: SMAJ5.0A, Diode_SMD:D_SMA, symbol Diode:SMAJ5.0A
- added D3: BZX84C10, Package_TO_SOT_SMD:SOT-23, symbol Device:D_Zener_Dual_CommonAnode_AKK_Split
- added J2: 1053131102, ROV_PCIe_USB_HUB:1053131102, symbol Connector:Screw_Terminal_01x02
- added J3: 691351500002, symbol Connector_Generic:Conn_01x02
- added Q1: DMP3018SFV, Package_SON:Diodes_PowerDI3333-8, symbol Transistor_FET:DMP3013SFV
- added R5: 100k, Resistor_SMD:R_0603_1608Metric, symbol Device:R_Small_US
- renumbered C58 to C1, R33 to R1, R1 to R2, R2 to R3, R3 to R4
Connections:
- net GND: now also D2.2 (A2), J2.1 (Pin_1), R5.2
- new net: D3.1 (A), D3.1 (A), Q1.4 (G), R5.1
- new net: D2.1 (A1), J2.2 (Pin_2), Q1.5 (D)
- new net VBUS: D3.3 (K), Q1.1 (S), Q1.2 (S), Q1.3 (S)
- no-connect marks 5 -> 8
Other:
- note added: "Receptacle: 1053131102"

Commit message: work
Parts:
- J3: value 691351500002 -> 1053071202; Part Number 691351500002 -> 1053071202
Other:
- note added: "Receptacle: 1053131102 Plug: 1053071202 Pins: 1053002100"
- note removed: "Receptacle: 1053131102"
Changed lines of the file:
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@@
 	(generator_version "10.0")
 	(paper "A4")
-	(text "Receptacle: 1053131102"
+	(text "Receptacle: 1053131102\nPlug:       1053071202\nPins:       1053002100"
 		(exclude_from_sim no)
 		(at 119.634 133.096 0)
@@
 			)
 		)
-		(property "Value" "691351500002"
+		(property "Value" "1053071202"
 			(at 140.97 142.2399 0)
 			(hide yes)
@@
 			)
 		)
-		(property "Part Number" "691351500002"
+		(property "Part Number" "1053071202"
 			(at 138.43 139.7 0)
 			(hide yes)

Commit message: changes
Other:
- moved on the sheet: J1, R2, R3, R4

Commit message: reroute
Parts:
- added J12: Raspberry_Pi_4, Connector_PinSocket_2.54mm:PinSocket_2x20_P2.54mm_Vertical, symbol Connector:Raspberry_Pi_4
Connections:
- net GND: now also J12.14 (GND), J12.20 (GND), J12.25 (GND), J12.30 (GND), J12.34 (GND), J12.39 (GND), J12.6 (GND), J12.9 (GND)
- new net: J12.1 (3V3), J12.17 (3V3)
- new net: J12.2 (5V), J12.4 (5V)
Other:
- moved on the sheet: C1, D1, D2, D3A, D3B, J2, J3, Q1, R1, R5
